File: power.kicad_sch (KiCad schematic)
At the start: 45 parts, among them J3 USB_C_Slave, U1 AP63200WU, U11 TPD2S300YFFR, U12 W25Q16JVSSIQ, U13 TPS65988DHRSHR, U14 AP63200WU, U15 TLV70012_SOT23-5

Commit message: Add files via upload
Parts:
- U3: renamed from U11; footprint Package_BGA:Texas_DSBGA-28_1.9x3mm_Layout4x7_P0.4mm -> Package_BGA:Texas_DSBGA-9_1.4715x1.4715mm_Layout3x3_P0.5mm
- renumbered C37 to C1, C40 to C10, C35 to C11, C41 to C12, C36 to C13, C52 to C14, C53 to C15, C29 to C16, C30 to C17, C6 to C18, C28 to C19, C32 to C2, C27 to C20, C26 to C21, C25 to C22, C38 to C3, C33 to C4, C21 to C5, C22 to C6, C1 to C7, C39 to C8, C34 to C9, D2 to D1, J3 to J1, L2 to L1, L1 to L2, R19 to R1, R15 to R10, R32 to R11, R33 to R12, R12 to R13, R18 to R2, R10 to R3, R11 to R4, R8 to R5, R9 to R6, R17 to R7, R13 to R8, R16 to R9, U14 to U1, U1 to U2, U15 to U4, U13 to U5, U12 to U6
Connections:
- net 3V3: now also U3.A2 (VBIAS); no longer U3.2 (VBIAS)
- net 5V: now also U3.C2 (VPWR); no longer U3.8 (VPWR)
- net CC1(2): now also U3.B1 (CC1); no longer U3.4 (CC1)
- net CC2(2): now also U3.B3 (CC2); no longer U3.6 (CC2)
- net C_CC1(2): now also U3.A1 (C_CC1); no longer U3.1 (C_CC1)
- net C_CC2(2): now also U3.A3 (C_CC2); no longer U3.3 (C_CC2)
- net GND: now also U3.B2 (GND), U3.C3 (VM); no longer U3.5 (GND), U3.9 (VM)
- net at R8.2: now also U3.C1 (FLT_N); no longer U3.7 (FLT_N)
