File: USB-C_3.2gen1.kicad_sch (KiCad schematic)
At the start: 5 parts, among them P1 USB_C_Plug_USB2.0

Commit message: Add files via upload
Parts:
- removed P1: USB_C_Plug_USB2.0, symbol Connector:USB_C_Plug_USB2.0
- removed R1, R2, R3, R4: R, symbol Device:R
Other:
- added sheet Block Diagram (block_diagram.kicad_sch)
- added sheet ETHERNET (ethernet.kicad_sch)
- added sheet HDMI (hdmi.kicad_sch)
- added sheet POWER (power.kicad_sch)
- added sheet SD (sd.kicad_sch)
- added sheet USB HUB (usb_hub.kicad_sch)
- added sheet USB-C MUX (usb-c_mux.kicad_sch)
- note added: "ETHERNET"
- note added: "HDMI"
- note added: "SD"
- note added: "USB HUB"
- note added: "USB-C Hub"
- note added: "USB-C MUX"
- note removed: "USB-C hub"
- title: (none) -> USB-C hub

Commit message: Add files via upload
Other:
- sheet HDMI renamed DisplayPort
- sheet DisplayPort: file hdmi.kicad_sch -> displayport.kicad_sch
- note added: "DisplayPort"
- note removed: "HDMI"
Changed lines of the file:
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@@
 		(date "2026-07-21")
 	)
-	(text "HDMI"
+	(text "DisplayPort"
 		(exclude_from_sim no)
 		(at 214.63 85.09 0)
@@
 			(color 72 72 72 1)
 		)
-		(property "Sheetname" "HDMI"
+		(property "Sheetname" "DisplayPort"
 			(at 165.481 88.5346 0)
 			(hide yes)
@@
 			)
 		)
-		(property "Sheetfile" "hdmi.kicad_sch"
+		(property "Sheetfile" "displayport.kicad_sch"
 			(at 149.479 94.885 0)
 			(hide yes)

Commit message: Add files via upload
Other:
- sheet POWER ports: added 1V2, 3V3, 5V, I2C_SCL, I2C_SDA, LDO_3V3, SYS_PWR, VBUS1, VBUS2; removed none
- sheet USB HUB ports: added 1V2, 3V3, 5V, GND, HUB_SSRX+, HUB_SSRX-, HUB_SSTX+, HUB_SSTX-, LAN_D+, LAN_D-, LAN_SSRX+, LAN_SSRX-, LAN_SSTX+, LAN_SSTX-, SD_D+, SD_D-, SD_SSRX+, SD_SSRX-, SD_SSTX+, SD_SSTX-, USB2_D+, USB2_D-, XTL0, XTLI; removed none

Commit message: Add files via upload
Other:
- sheet POWER ports: added none; removed 1V2, 3V3, 5V, I2C_SCL, I2C_SDA, LDO_3V3, SYS_PWR, VBUS1, VBUS2
- sheet USB HUB ports: added none; removed 1V2, 3V3, 5V, GND, HUB_SSRX+, HUB_SSRX-, HUB_SSTX+, HUB_SSTX-, LAN_D+, LAN_D-, LAN_SSRX+, LAN_SSRX-, LAN_SSTX+, LAN_SSTX-, SD_D+, SD_D-, SD_SSRX+, SD_SSRX-, SD_SSTX+, SD_SSTX-, USB2_D+, USB2_D-, XTL0, XTLI
