File: ethernet.kicad_sch (KiCad schematic)
At the start: 0 parts

Commit message: Add files via upload
Parts:
- added U5: RTL8152B-VB-CG, RTL8152B-VB-CG_RTK, symbol RTL8152B-VB-CG:RTL8152B-VB-CG
Changed lines of the file:
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@@
 		(date "2026-07-21")
 	)
+	(symbol
+		(lib_id "RTL8152B-VB-CG:RTL8152B-VB-CG")
+		(at 118.11 80.01 0)
+		(unit 1)
+		(body_style 1)
+		(exclude_from_sim no)
+		(in_bom yes)
+		(on_board yes)
+		(in_pos_files yes)
+		(dnp no)
+		(fields_autoplaced yes)
+		(property "Reference" "U5"
+			(at 156.21 69.85 0)
+			(show_name no)
+			(do_not_autoplace no)
+			(effects
+				(font
+					(size 1.524 1.524)
+				)
+			)
+		)
+		(property "Value" "RTL8152B-VB-CG"
+			(at 156.21 72.39 0)
+			(show_name no)
+			(do_not_autoplace no)
+			(effects
+				(font
+					(size 1.524 1.524)
+				)
+			)
+		)
+		(property "Footprint" "RTL8152B-VB-CG_RTK"
+			(at 118.11 80.01 0)
+			(hide yes)
+			(show_name no)
+			(do_not_autoplace no)
+			(effects
+				(font
+					(size 1.27 1.27)
+					(italic yes)
+				)
+			)
+		)
+		(property "Datasheet" "RTL8152B-VB-CG"
+			(at 118.11 80.01 0)
+			(hide yes)
+			(show_name no)
+			(do_not_autoplace no)
+			(effects
+				(font
+					(size 1.27 1.27)
+					(italic yes)
+				)
+			)
+		)
+		(property "Description" ""
+			(at 118.11 80.01 0)
+			(hide yes)
+			(show_name no)
+			(do_not_autoplace no)
+			(effects
+				(font
+					(size 1.27 1.27)
+				)
+			)
+		)
+		(pin "20"
+		)
+		(pin "25"
+		)
+		(pin "3"
+		)
+		(pin "17"
+		)
+		(pin "4"
+		)
+		(pin "18"
+		)
+		(pin "5"
+		)
+		(pin "6"
+		)
+		(pin "12"
+		)
+		(pin "13"
+		)
+		(pin "11"
+		)
+		(pin "7"
+		)
+		(pin "10"
+		)
+		(pin "9"
+		)
+		(pin "8"
+		)
+		(pin "2"
+		)
+		(pin "21"
+		)
+		(pin "1"
+		)
+		(pin "15"
+		)
+		(pin "22"
+		)
+		(pin "23"
+		)
+		(pin "24"
+		)
+		(pin "19"
+		)
+		(pin "14"
+		)
+		(pin "16"
+		)
+		(instances
+			(project "USB-C_3.2gen1"
+				(path "/d3213dd5-4179-4001-95f6-ec74c0d8f8ed/373a74f5-fd9e-49bb-a274-b26fbd7325a8"
+					(reference "U5")
+					(unit 1)
+				)
+			)
+		)
+	)
 )

Commit message: Add files via upload
Changed lines of the file:
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@@
 		(date "2026-07-21")
+	)
+	(wire
+		(pts
+			(xy 118.11 90.17) (xy 113.03 90.17)
+		)
+		(stroke
+			(width 0)
+			(type default)
+		)
+	)
+	(wire
+		(pts
+			(xy 118.11 87.63) (xy 113.03 87.63)
+		)
+		(stroke
+			(width 0)
+			(type default)
+		)
+	)
+	(wire
+		(pts
+			(xy 118.11 105.41) (xy 113.03 105.41)
+		)
+		(stroke
+			(width 0)
+			(type default)
+		)
+	)
+	(wire
+		(pts
+			(xy 118.11 102.87) (xy 113.03 102.87)
+		)
+		(stroke
+			(width 0)
+			(type default)
+		)
+	)
+	(wire
+		(pts
+			(xy 118.11 100.33) (xy 113.03 100.33)
+		)
+		(stroke
+			(width 0)
+			(type default)
+		)
+	)
+	(wire
+		(pts
+			(xy 194.31 90.17) (xy 200.66 90.17)
+		)
+		(stroke
+			(width 0)
+			(type default)
+		)
+	)
+	(wire
+		(pts
+			(xy 194.31 87.63) (xy 200.66 87.63)
+		)
+		(stroke
+			(width 0)
+			(type default)
+		)
+	)
+	(wire
+		(pts
+			(xy 194.31 92.71) (xy 200.66 92.71)
+		)
+		(stroke
+			(width 0)
+			(type default)
+		)
+	)
+	(wire
+		(pts
+			(xy 118.11 80.01) (xy 113.03 80.01)
+		)
+		(stroke
+			(width 0)
+			(type default)
+		)
+	)
+	(wire
+		(pts
+			(xy 194.31 85.09) (xy 200.66 85.09)
+		)
+		(stroke
+			(width 0)
+			(type default)
+		)
+	)
+	(wire
+		(pts
+			(xy 194.31 105.41) (xy 200.66 105.41)
+		)
+		(stroke
+			(width 0)
+			(type default)
+		)
+	)
+	(wire
+		(pts
+			(xy 194.31 100.33) (xy 200.66 100.33)
+		)
+		(stroke
+			(width 0)
+			(type default)
+		)
+	)
+	(wire
+		(pts
+			(xy 118.11 95.25) (xy 113.03 95.25)
+		)
+		(stroke
+			(width 0)
+			(type default)
+		)
+	)
+	(wire
+		(pts
+			(xy 118.11 82.55) (xy 113.03 82.55)
+		)
+		(stroke
+			(width 0)
+			(type default)
+		)
+	)
+	(wire
+		(pts
+			(xy 118.11 85.09) (xy 113.03 85.09)
+		)
+		(stroke
+			(width 0)
+			(type default)
+		)
+	)
+	(wire
+		(pts
+			(xy 118.11 107.95) (xy 113.03 107.95)
+		)
+		(stroke
+			(width 0)
+			(type default)
+		)
+	)
+	(wire
+		(pts
+			(xy 118.11 92.71) (xy 113.03 92.71)
+		)
+		(stroke
+			(width 0)
+			(type default)
+		)
+	)
+	(wire
+		(pts
+			(xy 194.31 80.01) (xy 200.66 80.01)
+		)
+		(stroke
+			(width 0)
+			(type default)
+		)
+	)
+	(wire
+		(pts
+			(xy 194.31 82.55) (xy 200.66 82.55)
+		)
+		(stroke
+			(width 0)
+			(type default)
+		)
+	)
+	(wire
+		(pts
+			(xy 194.31 95.25) (xy 200.66 95.25)
+		)
+		(stroke
+			(width 0)
+			(type default)
+		)
+	)
+	(wire
+		(pts
+			(xy 194.31 97.79) (xy 200.66 97.79)
+		)
+		(stroke
+			(width 0)
+			(type default)
+		)
+	)
+	(wire
+		(pts
+			(xy 118.11 97.79) (xy 113.03 97.79)
+		)
+		(stroke
+			(width 0)
+			(type default)
+		)
+	)
+	(wire
+		(pts
+			(xy 194.31 107.95) (xy 200.66 107.95)
+		)
+		(stroke
+			(width 0)
+			(type default)
+		)
+	)
+	(wire
+		(pts
+			(xy 194.31 102.87) (xy 200.66 102.87)
+		)
+		(stroke
+			(width 0)
+			(type default)
+		)
+	)
+	(wire
+		(pts
+			(xy 194.31 110.49) (xy 200.66 110.49)
+		)
+		(stroke
+			(width 0)
+			(type default)
+		)
 	)
 	(symbol

Commit message: Add files via upload
Parts:
- removed U5: RTL8152B-VB-CG, RTL8152B-VB-CG_RTK, symbol RTL8152B-VB-CG:RTL8152B-VB-CG
- added C69, C70, C73, C74, C75, C76, C77, C78, C80, C82, C83: 100nF, symbol Device:C_Small
- added C71, C72: 18pF, symbol Device:C_Small
- added C79: 4,7uF, symbol Device:C_Small
- added C81: 10nF, symbol Device:C_Small
- added J6: RJ45_JK0654219, Connector_RJ:RJ45_Pulse_JK0654219NL_Horizontal, symbol Connector:RJ45_JK0654219
- added R24: 2K49, symbol Device:R_Small
- added R25, R26: 330R, symbol Device:R_Small
- added R27: 1M, symbol Device:R_Small
- added U20: RTL8153B-VB-CG, RTL8153B-VB-CG:QFN40P500X500X90-41N, symbol RTL8153B-VB-CG:RTL8153B-VB-CG
- added Y2: 25MHz, symbol Device:Crystal_Small
Connections:
- new net: R24.2, U20.38 (RSET)
- new net: C81.1, J6.SH, R27.1
- new net: R26.1, U20.30 (EESK/LED1/SPISCK)
- new net: C69.2, U20.12 (U3SSTXN)
- new net: C70.2, U20.13 (U3SSTXP)
- new net: R25.1, U20.32 (LED0/SPICSB)
- new net: C80.1, J6.1 (MXCT3), J6.12 (MXCT1), J6.6 (MXCT2), J6.7 (MXCT4)
- new net 5V: U20.21 (VDD5), U20.27 (VDDREG5)
- new net AVDD10: C73.2, C74.2, C75.2, C76.2, C77.2, C78.1, C79.1, U20.14 (U3VDD10), U20.19 (U2VDD10), U20.22 (DVDD10_UPS), U20.28 (REGOUT), U20.3 (AVDD10), U20.34 (DVDD10), U20.37 (AVDD10), U20.8 (AVDD10)
- new net AVDD33: C82.1, C83.1, J6.14 (LED2+), J6.16 (LED1+), U20.11 (AVDD33), U20.20 (AVDD33), U20.23 (DVDD33), U20.26 (VDDREG33), U20.33 (DVDD33), U20.39 (AVDD33), U20.40 (AVDD33)
- new net CKXTAL1: C71.1, U20.35 (CKXTAL1), Y2.2
- new net CKXTAL2: C72.1, U20.36 (CKXTAL2), Y2.1
- new net GND: C71.2, C72.2, C73.1, C74.1, C75.1, C76.1, C77.1, C78.2, C79.2, C80.2, C81.2, C82.2, C83.2, R24.1, R27.2, U20.29 (GND), U20.41 (GND)
- new net LAN_D+: U20.18 (U2DP)
- new net LAN_D-: U20.17 (U2DM)
- new net LAN_SSRX+: U20.16 (U3SSRXP)
- new net LAN_SSRX-: U20.15 (U3SSRXN)
- new net LAN_SSTX+: C70.1
- new net LAN_SSTX-: C69.1
- new net LED0: J6.15 (LED1-), R25.2
- new net LED1: J6.13 (LED2-), R26.2
- new net MX1+: J6.11 (MX1+), U20.1 (MDIP0)
- new net MX1-: J6.10 (MX1-), U20.2 (MDIN0)
- new net MX2+: J6.4 (MX2+), U20.4 (MDIP1)
- new net MX2-: J6.5 (MX2-), U20.5 (MDIN1)
- new net MX3+: J6.3 (MX3+), U20.6 (MDIP2)
- new net MX3-: J6.2 (MX3-), U20.7 (MDIN2)
- new net MX4+: J6.8 (MX4+), U20.9 (MDIP3)
- new net MX4-: J6.9 (MX4-), U20.10 (MDIN3)
- no-connect marks 0 -> 3

Commit message: Add files via upload
Parts:
- added L3: 4,7uH, symbol Device:L_Small
Connections:
- net AVDD10: now also L3.2; no longer U20.28 (REGOUT)
- new net: L3.1, U20.28 (REGOUT)
Changed lines of the file:
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@@
 	)
 	(junction
-		(at 238.76 76.2)
+		(at 223.52 96.52)
 		(diameter 0)
 		(color 0 0 0 0)
 	)
 	(junction
-		(at 231.14 104.14)
+		(at 238.76 76.2)
 		(diameter 0)
 		(color 0 0 0 0)
 	)
 	(junction
-		(at 223.52 96.52)
+		(at 231.14 104.14)
 		(diameter 0)
 		(color 0 0 0 0)
@@
 	(wire
 		(pts
-			(xy 205.74 96.52) (xy 223.52 96.52)
-		)
-		(stroke
-			(width 0)
-			(type default)
-		)
-	)
-	(wire
-		(pts
 			(xy 91.44 104.14) (xy 106.68 104.14)
 		)
@@
 	(wire
 		(pts
+			(xy 220.98 96.52) (xy 223.52 96.52)
+		)
+		(stroke
+			(width 0)
+			(type default)
+		)
+	)
+	(wire
+		(pts
 			(xy 73.66 142.24) (xy 76.2 142.24)
 		)
@@
 	(wire
 		(pts
+			(xy 205.74 96.52) (xy 215.9 96.52)
+		)
+		(stroke
+			(width 0)
+			(type default)
+		)
+	)
+	(wire
+		(pts
 			(xy 124.46 71.12) (xy 121.92 71.12)
 		)
@@
 					(unit 1)
 				)
+			)
+		)
+	)
+	(symbol
+		(lib_id "Device:L_Small")
+		(at 218.44 96.52 90)
+		(unit 1)
+		(body_style 1)
+		(exclude_from_sim no)
+		(in_bom yes)
+		(on_board yes)
+		(in_pos_files yes)
+		(dnp no)
+		(fields_autoplaced yes)
+		(property "Reference" "L3"
+			(at 218.44 91.44 90)
+			(show_name no)
+			(do_not_autoplace no)
+			(effects
+				(font
+					(size 1.27 1.27)
+				)
+			)
+		)
+		(property "Value" "4,7uH"
+			(at 218.44 93.98 90)
+			(show_name no)
+			(do_not_autoplace no)
+			(effects
+				(font
+					(size 1.27 1.27)
+				)
+			)
+		)
+		(property "Footprint" ""
+			(at 218.44 96.52 0)
+			(hide yes)
+			(show_name no)
+			(do_not_autoplace no)
+			(effects
+				(font
+					(size 1.27 1.27)
+				)
+			)
+		)
+		(property "Datasheet" ""
+			(at 218.44 96.52 0)
+			(hide yes)
+			(show_name no)
+			(do_not_autoplace no)
+			(effects
+				(font
+					(size 1.27 1.27)
+				)
+			)
+		)
+		(property "Description" "Inductor, small symbol"
+			(at 218.44 96.52 0)
+			(hide yes)
+			(show_name no)
+			(do_not_autoplace no)
+			(effects
+				(font
+					(size 1.27 1.27)
+				)
+			)
+		)
+		(pin "1"
+		)
+		(pin "2"
+		)
+		(instances
+			(project "USB-C_3.2gen1"
+				(path "/d3213dd5-4179-4001-95f6-ec74c0d8f8ed/373a74f5-fd9e-49bb-a274-b26fbd7325a8"
+					(reference "L3")
+					(unit 1)
+				)

Commit message: Add files via upload
Parts:
- C69, C70, C71, C72, C73, C74, C75, C76, C77, C78, C80, C81, C82, C83: footprint (none) -> Capacitor_SMD:C_0603_1608Metric
- C79: footprint (none) -> Capacitor_SMD:C_1206_3216Metric
- L3, R24, R25, R26, R27: footprint (none) -> Resistor_SMD:R_0603_1608Metric
- Y2: footprint (none) -> Crystal:Crystal_SMD_3225-4Pin_3.2x2.5mm
Changed lines of the file:
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@@
 			)
 		)
-		(property "Footprint" ""
+		(property "Footprint" "Capacitor_SMD:C_0603_1608Metric"
 			(at 243.84 74.93 0)
 			(hide yes)
@@
 			)
 		)
-		(property "Footprint" ""
+		(property "Footprint" "Resistor_SMD:R_0603_1608Metric"
 			(at 128.27 96.52 0)
 			(hide yes)
@@
 			)
 		)
-		(property "Footprint" ""
+		(property "Footprint" "Capacitor_SMD:C_0603_1608Metric"
 			(at 121.92 76.2 0)
 			(hide yes)
@@
 			)
 		)
-		(property "Footprint" ""
+		(property "Footprint" "Capacitor_SMD:C_0603_1608Metric"
 			(at 76.2 138.43 0)
 			(hide yes)
@@
 			)
 		)
-		(property "Footprint" ""
+		(property "Footprint" "Capacitor_SMD:C_0603_1608Metric"
 			(at 132.08 76.2 0)
 			(hide yes)
@@
 			)
 		)
-		(property "Footprint" ""
+		(property "Footprint" "Resistor_SMD:R_0603_1608Metric"
 			(at 209.55 104.14 0)
 			(hide yes)
@@
 			)
 		)
-		(property "Footprint" ""
+		(property "Footprint" "Crystal:Crystal_SMD_3225-4Pin_3.2x2.5mm"
 			(at 127 71.12 0)
 			(hide yes)
@@
 			)
 		)
-		(property "Footprint" ""
+		(property "Footprint" "Capacitor_SMD:C_0603_1608Metric"
 			(at 227.33 129.54 0)
 			(hide yes)
@@
 			)
 		)
-		(property "Footprint" ""
+		(property "Footprint" "Capacitor_SMD:C_0603_1608Metric"
 			(at 222.25 76.2 0)
 			(hide yes)
@@
 			)
 		)
-		(property "Footprint" ""
+		(property "Footprint" "Capacitor_SMD:C_0603_1608Metric"
 			(at 228.6 68.58 0)
 			(hide yes)
@@
 			)
 		)
-		(property "Footprint" ""
+		(property "Footprint" "Capacitor_SMD:C_0603_1608Metric"
 			(at 228.6 81.28 0)
 			(hide yes)
@@
 			)
 		)
-		(property "Footprint" ""
+		(property "Footprint" "Capacitor_SMD:C_0603_1608Metric"
 			(at 231.14 100.33 0)
 			(hide yes)
@@
 			)
 		)
-		(property "Footprint" ""
+		(property "Footprint" "Capacitor_SMD:C_0603_1608Metric"
 			(at 243.84 82.55 0)
 			(hide yes)
@@
 			)
 		)
-		(property "Footprint" ""
+		(property "Footprint" "Capacitor_SMD:C_0603_1608Metric"
 			(at 222.25 83.82 0)
 			(hide yes)
@@
 			)
 		)
-		(property "Footprint" ""
+		(property "Footprint" "Capacitor_SMD:C_0603_1608Metric"
 			(at 228.6 73.66 0)
 			(hide yes)
@@
 			)
 		)
-		(property "Footprint" ""
+		(property "Footprint" "Resistor_SMD:R_0603_1608Metric"
 			(at 209.55 101.6 0)
 			(hide yes)
@@
 			)
 		)
-		(property "Footprint" ""
+		(property "Footprint" "Capacitor_SMD:C_0603_1608Metric"
 			(at 220.98 132.08 0)
 			(hide yes)
@@
 			)
 		)
-		(property "Footprint" ""
+		(property "Footprint" "Capacitor_SMD:C_0603_1608Metric"
 			(at 106.68 120.65 0)
 			(hide yes)
@@
 			)
 		)
-		(property "Footprint" ""
+		(property "Footprint" "Resistor_SMD:R_0603_1608Metric"
 			(at 218.44 96.52 0)
 			(hide yes)
@@
 			)
 		)
-		(property "Footprint" ""
+		(property "Footprint" "Capacitor_SMD:C_1206_3216Metric"
 			(at 223.52 100.33 0)
 			(hide yes)
@@
 			)
 		)
-		(property "Footprint" ""
+		(property "Footprint" "Resistor_SMD:R_0603_1608Metric"
 			(at 71.12 138.43 0)
 			(hide yes)

Commit message: Add files via upload
Other:
- moved on the sheet: C69, C70, C71, C72, C73, C74, C75, C76, C77, C78, C79, C80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

Commit message: Add files via upload
Parts:
- renumbered C81 to C67, C80 to C68, C71 to C69, C72 to C70, C69 to C71, C75 to C72, C77 to C73, C79 to C74, C70 to C75, C73 to C76, C74 to C77, C76 to C78, C78 to C79, C82 to C80, C83 to C81, R27 to R28, R24 to R29, R25 to R30, R26 to R31, U20 to U18
