File: sd.kicad_sch (KiCad schematic)
At the start: 0 parts

Commit message: Add files via upload
Parts:
- added U6: GL3224-ONY, Package_DFN_QFN:QFN-48-1EP_7x7mm_P0.5mm_EP5.15x5.15mm, symbol Interface_USB:GL3224-ONY
Connections:
- new net: U6.12 (GND), U6.3 (GND), U6.49 (GND)
- new net: U6.15 (AVDD33), U6.6 (AVDD33)
- new net: U6.25 (DVDD33), U6.34 (DVDD33), U6.44 (DVDD33)
Changed lines of the file:
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@@
 		(date "2026-07-21")
 	)
+	(symbol
+		(lib_id "Interface_USB:GL3224-ONY")
+		(at 158.75 97.79 0)
+		(unit 1)
+		(body_style 1)
+		(exclude_from_sim no)
+		(in_bom yes)
+		(on_board yes)
+		(in_pos_files yes)
+		(dnp no)
+		(fields_autoplaced yes)
+		(property "Reference" "U6"
+			(at 160.8933 143.51 0)
+			(show_name no)
+			(do_not_autoplace no)
+			(effects
+				(font
+					(size 1.27 1.27)
+				)
+				(justify left)
+			)
+		)
+		(property "Value" "GL3224-ONY"
+			(at 160.8933 146.05 0)
+			(show_name no)
+			(do_not_autoplace no)
+			(effects
+				(font
+					(size 1.27 1.27)
+				)
+				(justify left)
+			)
+		)
+		(property "Footprint" "Package_DFN_QFN:QFN-48-1EP_7x7mm_P0.5mm_EP5.15x5.15mm"
+			(at 156.21 151.384 0)
+			(hide yes)
+			(show_name no)
+			(do_not_autoplace no)
+			(effects
+				(font
+					(size 1.27 1.27)
+				)
+			)
+		)
+		(property "Datasheet" "https://lcsc.com/datasheet/lcsc_datasheet_2410121440_Genesys-Logic-GL3224-ONY04_C157358.pdf"
+			(at 156.21 153.67 0)
+			(hide yes)
+			(show_name no)
+			(do_not_autoplace no)
+			(effects
+				(font
+					(size 1.27 1.27)
+				)
+			)
+		)
+		(property "Description" "USB 3.0 Dual LUN Memory Card Reader Controller, external firmware support (SPI Flash Memory), WQFN-48"
+			(at 156.21 149.098 0)
+			(hide yes)
+			(show_name no)
+			(do_not_autoplace no)
+			(effects
+				(font
+					(size 1.27 1.27)
+				)
+			)
+		)
+		(pin "2"
+		)
+		(pin "1"
+		)
+		(pin "38"
+		)
+		(pin "49"
+		)
+		(pin "48"
+		)
+		(pin "47"
+		)
+		(pin "46"
+		)
+		(pin "39"
+		)
+		(pin "45"
+		)
+		(pin "44"
+		)
+		(pin "43"
+		)
+		(pin "42"
+		)
+		(pin "41"
+		)
+		(pin "40"
+		)
+		(pin "10"
+		)
+		(pin "9"
+		)
+		(pin "6"
+		)
+		(pin "4"
+		)
+		(pin "5"
+		)
+		(pin "7"
+		)
+		(pin "3"
+		)
+		(pin "8"
+		)
+		(pin "26"
+		)
+		(pin "37"
+		)
+		(pin "30"
+		)
+		(pin "33"
+		)
+		(pin "34"
+		)
+		(pin "28"
+		)
+		(pin "23"
+		)
+		(pin "31"
+		)
+		(pin "27"
+		)
+		(pin "35"
+		)
+		(pin "24"
+		)
+		(pin "22"
+		)
+		(pin "29"
+		)
+		(pin "25"
+		)
+		(pin "36"
+		)
+		(pin "32"
+		)
+		(pin "19"
+		)
+		(pin "17"
+		)
+		(pin "20"
+		)
+		(pin "16"
+		)
+		(pin "21"
+		)
+		(pin "18"
+		)
+		(pin "11"
+		)
+		(pin "12"
+		)
+		(pin "13"
+		)
+		(pin "14"
+		)
+		(pin "15"
+		)
+		(instances
+			(project "USB-C_3.2gen1"
+				(path "/d3213dd5-4179-4001-95f6-ec74c0d8f8ed/80a22beb-528f-4fff-8fe7-88006ebfcd3d"
+					(reference "U6")
+					(unit 1)
+				)
+			)
+		)
+	)
 )

Commit message: Add files via upload
Parts:
- added C84, C85: 18pF, symbol Device:C_Small
- added C86, C87, C88, C89, C90, C91, C94, C95: 100nF, symbol Device:C_Small
- added C92, C93: 10uF, symbol Device:C_Small
- added D3: Red, symbol Device:LED_Small
- added J7: 112L-TDA0, 112L-TDA0:CONN_112L-TDA0_ATT, symbol 112L-TDA0:112L-TDA0
- added J8: ST50S017VCAR1800, ST50S017VCAR1800:ST50S017VCAR1800_JAE, symbol ST50S017VCAR1800:ST50S017VCAR1800
- added R28: 10K, symbol Device:R_Small
- added R29: 330R, symbol Device:R_Small
- added Y3: 12MHz, symbol Device:Crystal_Small
Connections:
- net SD_SSRX-: now reaches U6.10 (RXN)
- net SD_SSRX+: now reaches U6.11 (RXP)
- net GND: now reaches U6.12 (GND), U6.3 (GND), U6.49 (GND)
- net GND: now also C84.2, C85.2, C88.2, C89.2, C90.2, C91.2, C92.2, C93.2, C94.2, C95.2, J7.10 (VSS), J7.13 (VSS), J7.16 (VSS), J7.19 (GND), J7.20 (GND), J7.21 (GND), J7.22 (GND), J7.23 (GND), J7.6 (VSS), R28.2, R29.2
- net X1: now reaches U6.13 (X1)
- net X1: now also C84.1, Y3.1
- net X2: now reaches U6.14 (X2)
- net X2: now also C85.1, Y3.2
- net 3V3: now reaches U6.15 (AVDD33), U6.6 (AVDD33)
- net 3V3: now also U6.24 (S2M2_VCC), U6.25 (DVDD33), U6.33 (VUHS_2), U6.34 (DVDD33), U6.44 (DVDD33), C88.1, C89.1, C92.1, C93.1, C94.1, C95.1, J7.4 (VDD), J7.9 (VDD2)
- net at U6.16 (RTERM): now also R28.1
- net at U6.21 (LED): now also D3.2 (A)
- net 5V: now reaches U6.22 (VBUS)
- net at U6.26 (DVDD12): now also C90.1
- net D1+: now reaches U6.27 (S2D1_M2BS)
- net D1+: now also J7.15 (D1+)
- net D1-: now reaches U6.28 (S2D0_M2D1)
- net D1-: now also J7.1 (DAT), J7.14 (D1-), J7.7 (DAT0)
- net D0+: now reaches U6.29 (S2CK_M2D0)
- net D0+: now also J7.11 (D0+)
- net D0-: now reaches U6.30 (S2CM_M2D2)
- net D0-: now also J7.12 (D0-)
- net DAT1: now reaches U6.31 (S2D3_M2D3)
- net DAT1: now also J7.8 (DAT1)
- net CLK: now reaches U6.32 (S2D2_M2CK)
- net CLK: now also J7.5 (CLK)
- net CD: now reaches U6.36 (SD2_CDZ)
- net CD: now also J7.18 (CD), J7.2 (CD/DAT3)
- net SD_D-: now reaches U6.4 (DM)
- net SD_D+: now reaches U6.5 (DP)
- net at U6.7 (TXN): now also C87.2
- net at U6.8 (TXP): now also C86.2
- net at U6.9 (AVDD12): now also C91.1
- new net: D3.1 (K), R29.1
- new net CMD: J7.3 (CMD)
- new net SD_SSTX+: C86.1
- new net SD_SSTX-: C87.1
- no-connect marks 0 -> 6

Commit message: Add files via upload
Parts:
- added C96, C97, C98, C99: 4,7uF, symbol Device:C_Small
- added R30: 10K, symbol Device:R_Small
- C93: value 10uF -> 100nF
- C94: value 100nF -> 10uF
- R28: value 10K -> 10K, 1%
Connections:
- net 3V3: now also C96.1, C97.1; no longer C92.1, C93.1, C94.1, C95.1, J7.4 (VDD), J7.9 (VDD2), U6.24 (S2M2_VCC), U6.33 (VUHS_2)
- net CLK: now also J8.5 (CLK), U6.39 (S1CK_M1D0); no longer J7.5 (CLK), U6.32 (S2D2_M2CK)
- net CMD: now also J8.3 (CMD), U6.40 (S1CM_M1D2); no longer J7.3 (CMD)
- net DAT1: now also J8.8 (DAT1RCLK-), U6.37 (S1D1_M1BS); no longer J7.8 (DAT1), U6.31 (S2D3_M2D3)
- net GND: now also J7.17 (SWIO), J8.10 (VSS), J8.13 (VSS), J8.16 (VSS), J8.6 (VSS), J8.DSW2, J8.GND1, J8.GND10, J8.GND2, J8.GND3, J8.GND4, J8.GND5, J8.GND6, J8.GND7, J8.GND8, J8.GND9, C96.2, C97.2, C98.2, C99.2, R30.2
- net SWIO: now reaches U6.1 (SD1_CDZ)
- net SWIO: now also J8.17 (SWIO)
- net DSW1: now reaches U6.2 (MS1_INS/SD1_WP)
- net DSW1: now also J8.DSW1
- net VDD: now reaches U6.23 (S1M1_VCC)
- net VDD: now also C94.1, C95.1, J8.4 (VDD1)
- net at C90.1, U6.26 (DVDD12): now also C98.1
- net at U6.35 (MS2_INS/SD2_WP): now also R30.1
- net DAT0: now reaches U6.38 (S1D0_M1D1)
- net DAT0: now also J8.7 (DAT0RCLK+)
- net DAT3: now reaches U6.41 (S1D3_M1D3)
- net DAT3: now also J8.2 (CD/DAT3)
- net DAT2: now reaches U6.42 (S1D2_M1CK)
- net DAT2: now also J8.1 (DAT2)
- net at C91.1, U6.9 (AVDD12): now also C99.1
- net CD renamed CD(2)
- net CD(2): no longer J7.2 (CD/DAT3)
- net D0+: no longer names the net of J7.11 (D0+)
- net D0+: no longer U6.29 (S2CK_M2D0)
- net D0-: no longer names the net of J7.12 (D0-)
- net D0-: no longer U6.30 (S2CM_M2D2)
- net D1+: no longer names the net of J7.15 (D1+)
- net D1+: no longer U6.27 (S2D1_M2BS)
- net D1- renamed DAT0(2)
- net DAT0(2): no longer J7.1 (DAT), J7.14 (D1-)
- new net CLK(2): J7.5 (CLK), U6.29 (S2CK_M2D0)
- new net CMD(2): J7.3 (CMD), U6.30 (S2CM_M2D2)
- new net DAT1(2): J7.8 (DAT1), U6.27 (S2D1_M2BS)
- new net DAT2(2): J7.1 (DAT), U6.32 (S2D2_M2CK)
- new net DAT3(2): J7.2 (CD/DAT3), U6.31 (S2D3_M2D3)
- new net VDD(2): C92.1, C93.1, J7.4 (VDD), U6.24 (S2M2_VCC)
- no-connect marks 6 -> 16
Other:
- moved on the sheet: C84, C85, C86, C87, C88, C89, C90, C91, D3, J7, J8, R28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

Commit message: Add files via upload
Parts:
- C84, C85, C86, C87, C88, C89, C90, C91, C93, C95: footprint (none) -> Capacitor_SMD:C_0603_1608Metric
- C92, C94, C96, C97, C98, C99: footprint (none) -> Capacitor_SMD:C_1206_3216Metric
- D3: footprint (none) -> LED_SMD:LED_0603_1608Metric
- R28, R29, R30: footprint (none) -> Resistor_SMD:R_0603_1608Metric
- Y3: footprint (none) -> Crystal:Crystal_SMD_3225-4Pin_3.2x2.5mm
Changed lines of the file:
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@@
 			)
 		)
-		(property "Footprint" ""
+		(property "Footprint" "Capacitor_SMD:C_0603_1608Metric"
 			(at 85.725 90.17 0)
 			(hide yes)
@@
 			)
 		)
-		(property "Footprint" ""
+		(property "Footprint" "Capacitor_SMD:C_1206_3216Metric"
 			(at 166.37 92.71 0)
 			(hide yes)
@@
 			)
 		)
-		(property "Footprint" ""
+		(property "Footprint" "Resistor_SMD:R_0603_1608Metric"
 			(at 154.94 149.86 0)
 			(hide yes)
@@
 			)
 		)
-		(property "Footprint" ""
+		(property "Footprint" "Capacitor_SMD:C_0603_1608Metric"
 			(at 170.18 92.71 0)
 			(hide yes)
@@
 			)
 		)
-		(property "Footprint" ""
+		(property "Footprint" "Capacitor_SMD:C_0603_1608Metric"
 			(at 128.27 55.88 0)
 			(hide yes)
@@
 			)
 		)
-		(property "Footprint" ""
+		(property "Footprint" "Capacitor_SMD:C_0603_1608Metric"
 			(at 79.375 87.63 0)
 			(hide yes)
@@
 			)
 		)
-		(property "Footprint" ""
+		(property "Footprint" "Capacitor_SMD:C_0603_1608Metric"
 			(at 78.74 68.58 0)
 			(hide yes)
@@
 			)
 		)
-		(property "Footprint" ""
+		(property "Footprint" "Resistor_SMD:R_0603_1608Metric"
 			(at 90.17 99.06 0)
 			(hide yes)
@@
 			)
 		)
-		(property "Footprint" ""
+		(property "Footprint" "Capacitor_SMD:C_0603_1608Metric"
 			(at 66.04 68.58 0)
 			(hide yes)
@@
 			)
 		)
-		(property "Footprint" ""
+		(property "Footprint" "Capacitor_SMD:C_1206_3216Metric"
 			(at 125.73 39.37 0)
 			(hide yes)
@@
 			)
 		)
-		(property "Footprint" ""
+		(property "Footprint" "Capacitor_SMD:C_1206_3216Metric"
 			(at 118.11 24.13 0)
 			(hide yes)
@@
 			)
 		)
-		(property "Footprint" ""
+		(property "Footprint" "Capacitor_SMD:C_0603_1608Metric"
 			(at 29.21 110.49 0)
 			(hide yes)
@@
 			)
 		)
-		(property "Footprint" ""
+		(property "Footprint" "Capacitor_SMD:C_1206_3216Metric"
 			(at 120.65 34.29 0)
 			(hide yes)
@@
 			)
 		)
-		(property "Footprint" ""
+		(property "Footprint" "Resistor_SMD:R_0603_1608Metric"
 			(at 160.02 125.73 0)
 			(hide yes)
@@
 			)
 		)
-		(property "Footprint" ""
+		(property "Footprint" "Capacitor_SMD:C_0603_1608Metric"
 			(at 120.65 29.21 0)
 			(hide yes)
@@
 			)
 		)
-		(property "Footprint" ""
+		(property "Footprint" "Capacitor_SMD:C_0603_1608Metric"
 			(at 118.11 20.32 0)
 			(hide yes)
@@
 			)
 		)
-		(property "Footprint" ""
+		(property "Footprint" "Crystal:Crystal_SMD_3225-4Pin_3.2x2.5mm"
 			(at 72.39 63.5 0)
 			(hide yes)
@@
 			)
 		)
-		(property "Footprint" ""
+		(property "Footprint" "LED_SMD:LED_0603_1608Metric"
 			(at 151.13 146.05 90)
 			(hide yes)
@@
 			)
 		)
-		(property "Footprint" ""
+		(property "Footprint" "Capacitor_SMD:C_1206_3216Metric"
 			(at 128.27 50.8 0)
 			(hide yes)
@@
 			)
 		)
-		(property "Footprint" ""
+		(property "Footprint" "Capacitor_SMD:C_1206_3216Metric"
 			(at 25.4 110.49 0)
 			(hide yes)
@@
 			)
 		)
-		(property "Footprint" ""
+		(property "Footprint" "Capacitor_SMD:C_0603_1608Metric"
 			(at 125.73 44.45 0)
 			(hide yes)

Commit message: Add files via upload
Other:
- moved on the sheet: C84, C85, C86, C87, C88, C89, C90, C91, C92, C93, C94, C95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

Commit message: Add files via upload
Parts:
- removed C94: 10uF, Capacitor_SMD:C_1206_3216Metric, symbol Device:C_Small
- removed C95: 100nF, Capacitor_SMD:C_0603_1608Metric, symbol Device:C_Small
- removed J8: ST50S017VCAR1800, ST50S017VCAR1800:ST50S017VCAR1800_JAE, symbol ST50S017VCAR1800:ST50S017VCAR1800
- added C96: 10uF, Capacitor_SMD:C_1206_3216Metric, symbol Device:C_Small
- added C97: 100nF, Capacitor_SMD:C_0603_1608Metric, symbol Device:C_Small
- added J8: 112L-TDA0, 112L-TDA0:CONN_112L-TDA0_ATT, symbol 112L-TDA0:112L-TDA0
- renumbered C92 to C82, C93 to C83, C87 to C86, C86 to C87, C91 to C88, C99 to C89, C98 to C91, C97 to C92, C89 to C93, C96 to C94, C88 to C95, R28 to R32, R29 to R33, R30 to R34, U6 to U19
Connections:
- net CLK: now also J8.5 (CLK)
- net CMD: now also J8.3 (CMD)
- net DAT0: now also J8.7 (DAT0)
- net DAT1: now also J8.8 (DAT1)
- net DAT2: now also J8.1 (DAT)
- net DAT3: now also J8.2 (CD/DAT3)
- net GND: now also C96.2, C97.2, J8.10 (VSS), J8.13 (VSS), J8.16 (VSS), J8.17 (SWIO), J8.19 (GND), J8.20 (GND), J8.21 (GND), J8.22 (GND), J8.23 (GND), J8.6 (VSS)
- net VDD: now also C96.1, C97.1, J8.4 (VDD)
- new net CD: J8.18 (CD)
- no-connect marks 16 -> 20
