File: usb-c_mux.kicad_sch (KiCad schematic)
At the start: 0 parts

Commit message: Add files via upload
Parts:
- added C1, C2, C3, C4, C5: 100nF, symbol Device:C_Small
- added C6: 10uF, symbol Device:C_Small
- added C7: 10nF, symbol Device:C_Small
- added J1: USB_C_Receptacle, symbol Connector:USB_C_Receptacle
- added R1, R2: 5K1, symbol Device:R_Small
- added R3: 1M, symbol Device:R_Small
- added U1: HD3SS3212IRKSR, HD3SS3212IRKSR:QFN50P450X250X100-21N, symbol HD3SS3212IRKSR:HD3SS3212IRKSR
- added U2, U3: TPD4E05U06DQA, Package_SON:USON-10_2.5x1.0mm_P0.5mm, symbol Power_Protection:TPD4E05U06DQA
Connections:
- new net: C7.2, J1.SH (SHIELD), R3.2
- new net: J1.A5 (CC1), R1.1
- new net: J1.B5 (CC2), R2.1
- new net 3V3: C1.1, C6.1, U1.6 (VCC)
- new net C0_N: C5.2, U1.14 (C0N)
- new net C0_P: C4.2, U1.15 (C0P)
- new net CC_ORIENT: U1.9 (SEL)
- new net EXP: C1.2, C6.2, C7.1, J1.A1 (GND), J1.A12 (GND), J1.B1 (GND), J1.B12 (GND), R1.2, R2.2, R3.1, U1.11 (GND), U1.2 (OEN), U1.20 (GND), U1.21 (EXP), U1.21_1 (EXP), U1.21_2 (EXP), U1.21_3 (EXP), U1.5 (GND), U2.3 (GND), U2.8 (GND), U3.3 (GND), U3.8 (GND)
- new net RX1+: J1.B11 (RX1+), U1.17 (B1P), U2.4 (D2+)
- new net RX1-: J1.B10 (RX1-), U1.16 (B1N), U2.5 (D2-)
- new net RX2+: J1.A11 (RX2+), U1.13 (C1P), U3.4 (D2+)
- new net RX2-: J1.A10 (RX2-), U1.12 (C1N), U3.5 (D2-)
- new net SBU1: J1.A8 (SBU1)
- new net SBU2: J1.B8 (SBU2)
- new net TX1+: C2.1, J1.A2 (TX1+), U2.1 (D1+)
- new net TX1-: C3.1, J1.A3 (TX1-), U2.2 (D1-)
- new net TX1_C_N: C3.2, U1.18 (B0N)
- new net TX1_C_P: C2.2, U1.19 (B0P)
- new net TX2+: C4.1, J1.B2 (TX2+), U3.1 (D1+)
- new net TX2-: C5.1, J1.B3 (TX2-), U3.2 (D1-)
- new net USB2_DN: J1.A7 (D-), J1.B7 (D-)
- new net USB2_DP: J1.A6 (D+), J1.B6 (D+)
- new net USB3_HUB_RX_N: U1.8 (A1N)
- new net USB3_HUB_RX_P: U1.7 (A1P)
- new net USB3_HUB_TX_N: U1.4 (A0N)
- new net USB3_HUB_TX_P: U1.3 (A0P)
- new net VBUS_5V: J1.A4 (VBUS), J1.A9 (VBUS), J1.B4 (VBUS), J1.B9 (VBUS)
- no-connect marks 0 -> 2

Commit message: Add files via upload
Parts:
- removed C1, C2, C3, C4, C5: 100nF, symbol Device:C_Small
- removed C6: 10uF, symbol Device:C_Small
- removed U1: HD3SS3212IRKSR, HD3SS3212IRKSR:QFN50P450X250X100-21N, symbol HD3SS3212IRKSR:HD3SS3212IRKSR
- added C10, C11, C12, C13, C14, C15, C16, C17, C8, C9: 100nF, symbol Device:C_Small
- added R4: 100K, symbol Device:R_Small
- added U7: TUSB546A-DCIRNQT, RNQ0040A, symbol TUSB546A-DCIRNQT:TUSB546A-DCIRNQT
- added U8: TPD4E05U06DQA, Package_SON:USON-10_2.5x1.0mm_P0.5mm, symbol Power_Protection:TPD4E05U06DQA
- added U9: USBLC6-2SC6, Package_TO_SOT_SMD:SOT-23-6, symbol Power_Protection:USBLC6-2SC6
- R1: value 5K1 -> 10K
- R2: value 5K1 -> 100K
Connections:
- net 3V3: now also R1.1, C10.1, C11.1, C8.1, C9.1, U7.1 (VCC), U7.20 (VCC), U7.28 (VCC), U7.6 (VCC)
- net RX1+: now also U7.30 (RX1P)
- net RX1-: now also U7.31 (RX1N)
- net RX2+: now also U7.40 (RX2P)
- net RX2-: now also U7.39 (RX2N)
- net SBU1: now also R4.2, U7.27 (SBU1)
- net SBU2: now also R2.2, U7.26 (SBU2)
- net TX1+: now also U7.33 (TX1P)
- net TX1-: now also U7.34 (TX1N)
- net TX2+: now also U7.37 (TX2P)
- net TX2-: now also U7.36 (TX2N)
- net VBUS_5V: now also U9.5 (VBUS)
- net at J1.A5 (CC1): no longer R1.1
- net at J1.B5 (CC2): no longer R2.1
- net EXP renamed GND
- net GND: now also R2.1, C10.2, C11.2, C8.2, C9.2, R4.1, U7.11 (SSEQ0_A0), U7.14 (DPEQ0_A1), U7.41 (PAD), U8.3 (GND), U8.8 (GND), U9.2 (GND); no longer R1.2, R2.2
- net USB2_DN renamed USB2*_D-
- net USB2*_D-: now also U9.1 (I/O1)
- net USB2_DP renamed USB2*_D+
- net USB2*_D+: now also U9.3 (I/O2)
- new net: C16.1, U7.12 (DP1P)
- new net: R1.2, U7.17 (I2C_EN)
- new net: C15.1, U7.10 (DP0N)
- new net: C17.1, U7.13 (DP1N)
- new net: C13.1, U7.8 (SSTXP)
- new net: C14.1, U7.9 (DP0P)
- new net: C12.1, U7.7 (SSTXN)
- new net DP_AUX+: U7.24 (AUXP)
- new net DP_AUX-: U7.25 (AUXN)
- new net DP_ML0+: C14.2, U8.1 (D1+)
- new net DP_ML0-: C15.2, U8.2 (D1-)
- new net DP_ML1+: C16.2, U8.4 (D2+)
- new net DP_ML1-: C17.2, U8.5 (D2-)
- new net HUB_SSRX+: U7.5 (SSRXP)
- new net HUB_SSRX-: U7.4 (SSRXN)
- new net HUB_SSTX+: C13.2
- new net HUB_SSTX-: C12.2
- new net I2C_SCL: U7.21 (FLIP_SCL)
- new net I2C_SDA: U7.22 (CTL0_SDA)
- new net MUX_HPD: U7.23 (CTL1_HPDIN)
- new net USB2_D+: U9.4 (I/O2)
- new net USB2_D-: U9.6 (I/O1)
- no-connect marks 2 -> 10
Other:
- moved on the sheet: C7, J1, R3, U2, U3

Commit message: Add files via upload
Parts:
- added C18: 1uF, symbol Device:C_Small
- added C19, C20: 100nF, symbol Device:C_Small
- added D1: SMAJ24A, Diode_SMD:D_SMA, symbol Diode:SMAJ24A
- added R5, R6, R7: 100K, symbol Device:R_Small
- added U10: TPD4S311YBFR, DSBGA16_1P69X1P69_TEX, symbol TPD4S311YBFR:TPD4S311YBFR
- J1: value USB_C_Receptacle -> USB_C_Master
- R2, R4: value 100K -> 2M
Connections:
- net 3V3: now also C18.2, R5.2, R7.1, U10.C4 (VPWR)
- net DP_AUX+: now also R6.2
- net DP_AUX-: now also R5.1
- net GND: now also C18.1, C19.2, C20.1, D1.2 (A2), R6.1, U10.C1 (GND), U10.C2 (GND), U10.C3 (GND)
- net SBU1: now also U10.D1 (SBU1); no longer J1.A8 (SBU1)
- net SBU2: now also U10.D2 (SBU2); no longer J1.B8 (SBU2)
- net C_CC1: now reaches J1.A5 (CC1)
- net C_CC1: now also U10.A2 (C_CC1)
- net C_CC2: now reaches J1.B5 (CC2)
- net C_CC2: now also U10.A3 (C_CC2)
- net VBUS_5V renamed VBUS
- net VBUS: now also D1.1 (A1); no longer U9.5 (VBUS)
- new net: C19.1, U10.A4 (VBIAS)
- new net: R7.2, U10.B4 (FLT)
- new net 5V: C20.2, U9.5 (VBUS)
- new net CC1: U10.D3 (CC1)
- new net CC2: U10.D4 (CC2)
- new net SBU*1: J1.A8 (SBU1), U10.B1 (C_SBU1)
- new net SBU*2: J1.B8 (SBU2), U10.A1 (C_SBU2)
- no-connect marks 10 -> 12
Other:
- moved on the sheet: U2, U3, U8, U9

Commit message: Add files via upload
Connections:
- net VBUS renamed VBUS2
Other:
- note added: "SEARCHING"
Changed lines of the file:
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@@
 		(date "2026-07-21")
+	)
+	(text "SEARCHING"
+		(exclude_from_sim no)
+		(at 383.794 100.584 0)
+		(effects
+			(font
+				(size 12.7 12.7)
+				(thickness 2.54)
+				(bold yes)
+			)
+		)
 	)
 	(junction
@@
 		)
 	)
-	(hierarchical_label "VBUS"
+	(hierarchical_label "VBUS2"
 		(shape input)
 		(at 55.88 27.94 0)

Commit message: Add files via upload
Other:
- moved on the sheet: R5
Changed lines of the file:
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@@
 	)
 	(junction
+		(at 93.98 77.47)
+		(diameter 0)
+		(color 0 0 0 0)
+	)
+	(junction
 		(at 92.71 154.94)
 		(diameter 0)
@@
 	)
 	(junction
-		(at 96.52 77.47)
-		(diameter 0)
-		(color 0 0 0 0)
-	)
-	(junction
 		(at 53.34 55.88)
 		(diameter 0)
@@
 	)
 	(no_connect
-		(at 102.87 87.63)
+		(at 111.76 59.69)
 	)
 	(no_connect
-		(at 102.87 67.31)
+		(at 111.76 87.63)
 	)
 	(no_connect
-		(at 175.26 100.33)
+		(at 111.76 69.85)
 	)
 	(no_connect
-		(at 36.83 152.4)
+		(at 167.64 100.33)
 	)
 	(no_connect
-		(at 102.87 69.85)
+		(at 41.91 152.4)
 	)
 	(no_connect
-		(at 102.87 62.23)
+		(at 111.76 62.23)
 	)
 	(no_connect
-		(at 175.26 52.07)
+		(at 167.64 52.07)
 	)
 	(no_connect
-		(at 36.83 149.86)
+		(at 41.91 149.86)
 	)
 	(no_connect
-		(at 102.87 59.69)
+		(at 111.76 67.31)
 	)
 	(no_connect
-		(at 175.26 95.25)
+		(at 167.64 95.25)
 	)
 	(no_connect
-		(at 175.26 102.87)
+		(at 167.64 102.87)
 	)
 	(no_connect
-		(at 175.26 64.77)
-	)
-	(wire
-		(pts
-			(xy 111.76 69.85) (xy 102.87 69.85)
-		)
-		(stroke
-			(width 0)
-			(type default)
-		)
+		(at 167.64 64.77)
 	)
 	(wire
@@
 	(wire
 		(pts
-			(xy 54.61 181.61) (xy 58.42 181.61)
+			(xy 93.98 77.47) (xy 111.76 77.47)
 		)
 		(stroke
@@
 	(wire
 		(pts
-			(xy 109.22 181.61) (xy 114.3 181.61)
+			(xy 54.61 181.61) (xy 58.42 181.61)
 		)
 		(stroke
@@
 	(wire
 		(pts
-			(xy 105.41 82.55) (xy 100.33 82.55)
+			(xy 109.22 181.61) (xy 114.3 181.61)
 		)
 		(stroke
@@
 	(wire
 		(pts
-			(xy 111.76 67.31) (xy 102.87 67.31)
+			(xy 105.41 82.55) (xy 100.33 82.55)
 		)
 		(stroke
@@
 	(wire
 		(pts
-			(xy 96.52 67.31) (xy 96.52 66.04)
+			(xy 87.63 147.32) (xy 101.6 147.32)
 		)
 		(stroke
@@
 	(wire
 		(pts
-			(xy 87.63 147.32) (xy 101.6 147.32)
+			(xy 93.98 77.47) (xy 91.44 77.47)
 		)
 		(stroke
@@
 	(wire
 		(pts
-			(xy 111.76 87.63) (xy 102.87 87.63)
-		)
-		(stroke
-			(width 0)
-			(type default)
-		)
-	)
-	(wire
-		(pts
 			(xy 161.29 181.61) (xy 165.1 181.61)
 		)
@@
 	(wire
 		(pts
-			(xy 167.64 64.77) (xy 175.26 64.77)
+			(xy 93.98 60.96) (xy 93.98 66.04)
 		)
 		(stroke
@@
 	(wire
 		(pts
-			(xy 96.52 77.47) (xy 91.44 77.47)
-		)
-		(stroke
-			(width 0)
-			(type default)
-		)
-	)
-	(wire
-		(pts
 			(xy 49.53 68.58) (xy 53.34 68.58)
 		)
@@
 	(wire
 		(pts
-			(xy 111.76 59.69) (xy 102.87 59.69)
-		)
-		(stroke
-			(width 0)
-			(type default)
-		)
-	)
-	(wire
-		(pts
 			(xy 101.6 147.32) (xy 101.6 149.86)
 		)
@@
 	(wire
 		(pts
-			(xy 167.64 95.25) (xy 175.26 95.25)
-		)
-		(stroke
-			(width 0)
-			(type default)
-		)
-	)
-	(wire
-		(pts
 			(xy 26.67 101.6) (xy 26.67 105.41)
 		)
@@
 	(wire
 		(pts
-			(xy 167.64 52.07) (xy 175.26 52.07)
-		)
-		(stroke
-			(width 0)
-			(type default)
-		)
-	)
-	(wire
-		(pts
 			(xy 111.76 107.95) (xy 102.87 107.95)
 		)
@@
 	(wire
 		(pts
-			(xy 111.76 77.47) (xy 96.52 77.47)
-		)
-		(stroke
-			(width 0)
-			(type default)
-		)
-	)
-	(wire
-		(pts
 			(xy 49.53 78.74) (xy 53.34 78.74)
 		)
@@
 	(wire
 		(pts
-			(xy 167.64 100.33) (xy 175.26 100.33)
-		)
-		(stroke
-			(width 0)
-			(type default)
-		)
-	)
-	(wire
-		(pts
 			(xy 26.67 113.03) (xy 34.29 113.03)
 		)
@@
 	(wire
 		(pts
-			(xy 167.64 102.87) (xy 175.26 102.87)
-		)
-		(stroke
-			(width 0)
-			(type default)
-		)
-	)
-	(wire
-		(pts
 			(xy 110.49 44.45) (xy 111.76 44.45)
 		)
@@
 	(wire
 		(pts
-			(xy 96.52 66.04) (xy 95.25 66.04)
-		)
-		(stroke
-			(width 0)
-			(type default)
-		)
-	)
-	(wire
-		(pts
 			(xy 167.64 46.99) (xy 175.26 46.99)
 		)
@@
 	(wire
 		(pts
-			(xy 111.76 62.23) (xy 102.87 62.23)
-		)
-		(stroke
-			(width 0)
-			(type default)
-		)
-	)
-	(wire
-		(pts
 			(xy 102.87 105.41) (xy 102.87 107.95)
 		)
@@
 	(wire
 		(pts
-			(xy 41.91 152.4) (xy 36.83 152.4)
-		)
-		(stroke
-			(width 0)
-			(type default)
-		)
-	)
-	(wire
-		(pts
 			(xy 41.91 147.32) (xy 36.83 147.32)
 		)
@@
 	(wire
 		(pts
-			(xy 96.52 72.39) (xy 96.52 77.47)
+			(xy 93.98 71.12) (xy 93.98 77.47)
 		)
 		(stroke
@@
 	(wire
 		(pts
-			(xy 41.91 149.86) (xy 36.83 149.86)
-		)
-		(stroke
-			(width 0)
-			(type default)
-		)
-	)
-	(wire
-		(pts
 			(xy 167.64 74.93) (xy 193.04 74.93)
 		)
@@
 	(hierarchical_label "3V3"
 		(shape input)
-		(at 95.25 66.04 180)
+		(at 93.98 60.96 180)
 		(effects
 			(font
@@
 	(symbol
 		(lib_id "Device:R_Small")
-		(at 96.52 69.85 180)
+		(at 93.98 68.58 180)
 		(unit 1)
 		(body_style 1)
@@
 		(dnp no)
 		(property "Reference" "R5"
-			(at 99.568 71.12 0)
+			(at 98.298 67.31 0)
 			(show_name no)
 			(do_not_autoplace no)
@@
 		)
 		(property "Value" "100K"
-			(at 99.822 69.342 0)
+			(at 98.044 69.088 0)
 			(show_name no)
 			(do_not_autoplace no)
@@
 		)
 		(property "Footprint" ""
-			(at 96.52 69.85 0)
+			(at 93.98 68.58 0)
 			(hide yes)
 			(show_name no)
@@
 		)
 		(property "Datasheet" ""
-			(at 96.52 69.85 0)
+			(at 93.98 68.58 0)
 			(hide yes)
 			(show_name no)
@@
 		)
 		(property "Description" "Resistor, small symbol"
-			(at 96.52 69.85 0)
+			(at 93.98 68.58 0)
 			(hide yes)
 			(show_name no)

Commit message: Add files via upload
Parts:
- removed C11: 100nF, symbol Device:C_Small
- removed U7: TUSB546A-DCIRNQT, RNQ0040A, symbol TUSB546A-DCIRNQT:TUSB546A-DCIRNQT
- added R34: 10K, Resistor_SMD:R_0603_1608Metric, symbol Device:R_Small
- added U5: TUSB564IRNQR, Package_DFN_QFN:Texas_RNQ0040A_WQFN-40-1EP_6x4mm_P0.4mm_EP4.7x2.7mm_ThermalVias, symbol TUSB564IRNQR:TUSB564IRNQR
- C10, C12, C13, C14, C15, C16, C17, C18, C19, C20, C7, C8, C9: footprint (none) -> Capacitor_SMD:C_0603_1608Metric
- J1: footprint (none) -> Connector_USB:USB_C_Receptacle_Molex_105450-0101
- R1, R2, R3, R4, R5, R6, R7: footprint (none) -> Resistor_SMD:R_0603_1608Metric
- U10: footprint DSBGA16_1P69X1P69_TEX -> Package_BGA:Texas_YFP0020_DSBGA-20_1.588x1.988mm_Layout4x5_P0.4mm
Connections:
- net 3V3: now also R34.1, U5.28 (VCC); no longer C8.1, C9.1
- net DP_AUX+: now also U5.26 (AUXP)
- net DP_AUX-: now also U5.27 (AUXN)
- net GND: now also U5.35 (DPEQ0_A1), U5.38 (SSEQ0_A0), U5.41 (GND)
- net HUB_SSRX+: now also U5.8 (SSTXP)
- net HUB_SSRX-: now also U5.7 (SSTXN)
- net I2C_SCL: now also U5.21 (FLIP_SCL)
- net I2C_SDA: now also U5.22 (CTL0_SDA)
- net MUX_HPD: now also U5.32 (HPDIN)
- net RX1+: now also U5.12 (RX1P)
- net RX1-: now also U5.13 (RX1N)
- net RX2+: now also U5.16 (RX2P)
- net RX2-: now also U5.15 (RX2N)
- net SBU1: now also U5.24 (SBU1)
- net SBU2: now also U5.25 (SBU2)
- net TX1+: now also U5.9 (TX1P)
- net TX1-: now also U5.10 (TX1N)
- net TX2+: now also U5.19 (TX2P)
- net TX2-: now also U5.18 (TX2N)
- net at C16.1: now also U5.37 (DP1P)
- net at R1.2: now also U5.17 (I2C_EN)
- net at C15.1: now also U5.39 (DP0N)
- net at C17.1: now also U5.36 (DP1N)
- net at C13.1: now also U5.5 (SSRXP)
- net at C14.1: now also U5.40 (DP0P)
- net at C12.1: now also U5.4 (SSRXN)
- new net: C8.1, U5.6 (VCC)
- new net: C9.1, U5.20 (VCC)
- new net: R34.2, U5.29 (EN)
Other:
- note added: "ASSIGNING FOOTPRINTS"
- note removed: "SEARCHING"
- moved on the sheet: C10, C12, C13, C14, C15, C16, C17, C8, C9, R1, R2, R4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

Commit message: Add files via upload
Other:
- moved on the sheet: C10, C12, C13, C14, C15, C16, C17, C18, C19, C20, C7, C8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

Commit message: Add files via upload
Parts:
- U7: renamed from U10; footprint Package_BGA:Texas_YFP0020_DSBGA-20_1.588x1.988mm_Layout4x5_P0.4mm -> Package_BGA:Texas_DSBGA-16_2.39x2.39mm_Layout4x4_P0.5mm
- renumbered C7 to C23, C19 to C24, C18 to C25, C10 to C26, C9 to C27, C8 to C28, C20 to C29, C14 to C30, C16 to C31, C12 to C32, C13 to C33, C15 to C34, C17 to C35, D1 to D2, J1 to J2, R3 to R14, R7 to R15, R2 to R16, R4 to R17, R34 to R18, R1 to R19, R5 to R20, R6 to R21, U9 to U10, U2 to U11, U5 to U12, U3 to U9
