File: usb_hub.kicad_sch (KiCad schematic)
At the start: 0 parts

Commit message: Add files via upload
Parts:
- added U4: RTS5411-GRT, QFN76_RTK, symbol ul_RTS5411-GRT:RTS5411-GRT

Commit message: Add files via upload
Parts:
- added C2: 1uF, symbol Device:C_Small
- added C23, C24, C3, C4, C42, C43, C44, C45, C46, C47, C5: 100nF, symbol Device:C_Small
- added C48, C49: 18pF, symbol Device:C_Small
- added R14: 12K1, symbol Device:R_Small
- added Y1: 24MHz, symbol Device:Crystal_Small
Connections:
- net at U4.1 (RREF): now also R14.2
- net at U4.13 (AV12): now also C24.2
- net at U4.19 (AV12): now also C42.2
- net 3V3: now reaches U4.22 (DV33)
- net 3V3: now also U4.4 (DV33), U4.48 (DV33), U4.73 (DV33)
- net at U4.25 (AV12): now also C43.2
- net at U4.3 (DV12): now also C3.1
- net at U4.31 (AV12): now also C44.2
- net at U4.49 (DV12): now also C5.1
- net at U4.50 (DV12): now also C4.1
- net GND: now reaches U4.51 (GND)
- net GND: now also U4.61 (GND), U4.77 (REFGND), C2.1, C23.1, C24.1, C3.2, C4.2, C42.1, C43.1, C44.1, C45.1, C46.1, C47.1, C48.2, C49.2, C5.2, R14.1
- net 5V: now reaches U4.53 (LDO_V5_IN)
- net 5V: now also U4.54 (LDO_V5_IN)
- net at U4.55 (V33_OUT): now also C2.2
- net at U4.58 (AV12): now also C47.2
- net at U4.64 (AV12): now also C46.2
- net at U4.7 (AV12): now also C23.2
- net at U4.70 (AV12): now also C45.2
- net XTLI: now reaches U4.74 (XTLI)
- net XTLI: now also C49.1, Y1.2
- net XTL0: now reaches U4.75 (XTLO)
- net XTL0: now also C48.1, Y1.1

Commit message: Add files via upload
Parts:
- added C50, C51, C54, C55, C56, C57, C58, C59, C60, C61, C62, C63, C64, C65, C66, C67: 100nF, symbol Device:C_Small
- added C68: 10uF, symbol Device:C_Small
- added F1: 1,5A, symbol Device:Polyfuse_Small
- added J4: USB3_A, symbol Connector:USB3_A
- added J5: USB_C_Receptacle, Connector_USB:USB_C_Receptacle_Molex_105450-0101, symbol Connector:USB_C_Receptacle
- added R20, R21: 10K, symbol Device:R_Small
- added R22, R23: 56K, symbol Device:R_Small
- added U16, U17: USBLC6-2SC6, Package_TO_SOT_SMD:SOT-23-6, symbol Power_Protection:USBLC6-2SC6
- added U18, U19: TPD4E05U06DQA, Package_SON:USON-10_2.5x1.0mm_P0.5mm, symbol Power_Protection:TPD4E05U06DQA
Connections:
- net 3V3: now also U4.2 (BPWR_DET), U4.76 (SPWR_DET), R20.2, R21.2
- net 5V: now also C62.2, C63.2, C68.1, F1.2, J5.A4 (VBUS), J5.A9 (VBUS), J5.B4 (VBUS), J5.B9 (VBUS), R22.2, R23.2, U16.5 (VBUS), U17.5 (VBUS)
- net GND: now also C62.1, C63.1, C68.2, J4.4 (GND), J4.7 (DRAIN), J4.SH (SHIELD), J5.A1 (GND), J5.A12 (GND), J5.B1 (GND), J5.B12 (GND), J5.SH (SHIELD), U16.2 (GND), U17.2 (GND), U18.3 (GND), U18.8 (GND), U19.3 (GND), U19.8 (GND)
- net 1V2: now reaches C4.1, U4.50 (DV12)
- net 1V2: now also C23.2, C24.2, C3.1, C42.2, C43.2, C44.2, C45.2, C46.2, C47.2, C5.1, U4.13 (AV12), U4.19 (AV12), U4.25 (AV12), U4.3 (DV12), U4.31 (AV12), U4.49 (DV12), U4.58 (AV12), U4.64 (AV12), U4.7 (AV12), U4.70 (AV12)
- net at U4.10 (OCP2): now also R20.1
- net SD_SSTX+: now reaches U4.11 (DSP2_SSRX+)
- net SD_SSTX-: now reaches U4.12 (DSP2_SSRX-)
- net at U4.14 (DSP3_SSTX+): now also C58.2
- net at U4.15 (DSP3_SSTX-): now also C59.2
- net USBA_SSTX+: now reaches U4.17 (DSP3_SSRX+)
- net USBA_SSTX+: now also C64.1, U18.1 (D1+)
- net USBA_SSTX-: now reaches U4.18 (DSP3_SSRX-)
- net USBA_SSTX-: now also C65.1, U18.2 (D1-)
- net USBA_D+: now reaches U4.20 (DSP3_DP)
- net USBA_D+: now also U16.4 (I/O2)
- net USBA_D-: now reaches U4.21 (DSP3_DM)
- net USBA_D-: now also U16.6 (I/O1)
- net USBC_D+: now reaches U4.23 (DSP4_DP)
- net USBC_D+: now also U17.6 (I/O1)
- net USBC_D-: now reaches U4.24 (DSP4_DM)
- net USBC_D-: now also U17.4 (I/O2)
- net at U4.26 (DSP4_SSTX+): now also C60.2
- net at U4.27 (DSP4_SSTX-): now also C61.2
- net USBC_SSTX+: now reaches U4.29 (DSP4_SSRX-)
- net USBC_SSTX+: now also C66.1, U19.4 (D2+)
- net USBC_SSTX-: now reaches U4.30 (DSP4_SSRX+)
- net USBC_SSTX-: now also C67.1, U19.5 (D2-)
- net SD_D+: now reaches U4.5 (DSP2_DP)
- net USB2_D+: now reaches U4.56 (USP_DP)
- net USB2_D-: now reaches U4.57 (USP_DM)
- net at U4.59 (USP_SSTX-): now also C50.2
- net SD_D-: now reaches U4.6 (DSP2_DM)
- net at U4.60 (USP_SSTX+): now also C51.2
- net HUB_SSTX-: now reaches U4.62 (USP_SSRX-)
- net HUB_SSTX+: now reaches U4.63 (USP_SSRX+)
- net at U4.65 (DSP1_SSTX+): now also C54.2
- net at U4.66 (DSP1_SSTX-): now also C55.2
- net at U4.67 (OCP1): now also R21.1
- net LAN_SSTX+: now reaches U4.68 (DSP1_SSRX+)
- net LAN_SSTX-: now reaches U4.69 (DSP1_SSRX-)
- net LAN_D+: now reaches U4.71 (DSP1_DP)
- net LAN_D-: now reaches U4.72 (DSP1_DM)
- net at U4.8 (DSP2_SSTX+): now also C57.2
- net at U4.9 (DSP2_SSTX-): now also C56.2
- new net: C65.2, J4.8 (SSTX-)
- new net: J5.A5 (CC1), R22.1
- new net: C66.2, J5.A2 (TX1+)
- new net: C67.2, J5.A3 (TX1-)
- new net: J5.B5 (CC2), R23.1
- new net: C64.2, J4.9 (SSTX+)
- new net: F1.1, J4.1 (VBUS)
- new net HUB_SSRX+: C51.1
- new net HUB_SSRX-: C50.1
- new net LAN_SSRX+: C54.1
- new net LAN_SSRX-: C55.1
- new net SD_SSRX+: C57.1
- new net SD_SSRX-: C56.1
- new net USBA_*D+: J4.3 (D+), U16.3 (I/O2)
- new net USBA_*D-: J4.2 (D-), U16.1 (I/O1)
- new net USBA_SSRX+: C58.1, J4.6 (SSRX+), U18.4 (D2+)
- new net USBA_SSRX-: C59.1, J4.5 (SSRX-), U18.5 (D2-)
- new net USBC_*D+: J5.A6 (D+), J5.B6 (D+), U17.1 (I/O1)
- new net USBC_*D-: J5.A7 (D-), J5.B7 (D-), U17.3 (I/O2)
- new net USBC_SSRX+: C60.1, J5.B11 (RX1+), U19.1 (D1+)
- new net USBC_SSRX-: C61.1, J5.B10 (RX1-), U19.2 (D1-)
- no-connect marks 0 -> 24
Other:
- moved on the sheet: C2, C23, C24, C3, C4, C42, C43, C44, C45, C46, C47, C48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

Commit message: Add files via upload
Parts:
- added R31: 1M, symbol Device:R_Small
Connections:
- net XTL0: now also R31.2
- net XTLI: now also R31.1
Other:
- moved on the sheet: C48, C49
Changed lines of the file:
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@@
 	)
 	(junction
-		(at 274.32 113.03)
-		(diameter 0)
-		(color 0 0 0 0)
-	)
-	(junction
 		(at 99.06 102.87)
 		(diameter 0)
@@
 	)
 	(junction
-		(at 269.24 121.92)
+		(at 264.16 113.03)
 		(diameter 0)
 		(color 0 0 0 0)
 	)
 	(junction
-		(at 264.16 113.03)
+		(at 264.16 116.84)
+		(diameter 0)
+		(color 0 0 0 0)
+	)
+	(junction
+		(at 269.24 124.46)
+		(diameter 0)
+		(color 0 0 0 0)
+	)
+	(junction
+		(at 274.32 113.03)
+		(diameter 0)
+		(color 0 0 0 0)
+	)
+	(junction
+		(at 274.32 116.84)
 		(diameter 0)
 		(color 0 0 0 0)
@@
 	(wire
 		(pts
-			(xy 264.16 121.92) (xy 269.24 121.92)
+			(xy 264.16 124.46) (xy 269.24 124.46)
 		)
 		(stroke
@@
 	(wire
 		(pts
-			(xy 264.16 113.03) (xy 264.16 115.57)
+			(xy 264.16 113.03) (xy 264.16 116.84)
 		)
 		(stroke
@@
 	(wire
 		(pts
-			(xy 274.32 121.92) (xy 274.32 120.65)
+			(xy 274.32 124.46) (xy 274.32 123.19)
 		)
 		(stroke
@@
 	(wire
 		(pts
-			(xy 274.32 113.03) (xy 274.32 115.57)
+			(xy 274.32 113.03) (xy 274.32 116.84)
 		)
 		(stroke
@@
 	(wire
 		(pts
+			(xy 271.78 116.84) (xy 274.32 116.84)
+		)
+		(stroke
+			(width 0)
+			(type default)
+		)
+	)
+	(wire
+		(pts
 			(xy 274.32 113.03) (xy 275.59 113.03)
 		)
@@
 	(wire
 		(pts
-			(xy 269.24 121.92) (xy 269.24 123.19)
+			(xy 269.24 124.46) (xy 269.24 125.73)
 		)
 		(stroke
@@
 	(wire
 		(pts
-			(xy 264.16 120.65) (xy 264.16 121.92)
+			(xy 264.16 123.19) (xy 264.16 124.46)
 		)
 		(stroke
@@
 	(wire
 		(pts
+			(xy 264.16 116.84) (xy 264.16 118.11)
+		)
+		(stroke
+			(width 0)
+			(type default)
+		)
+	)
+	(wire
+		(pts
 			(xy 149.86 44.45) (xy 148.59 44.45)
 		)
@@
 	(wire
 		(pts
+			(xy 274.32 116.84) (xy 274.32 118.11)
+		)
+		(stroke
+			(width 0)
+			(type default)
+		)
+	)
+	(wire
+		(pts
 			(xy 96.52 135.89) (xy 100.33 135.89)
 		)
@@
 	(wire
 		(pts
+			(xy 264.16 116.84) (xy 266.7 116.84)
+		)
+		(stroke
+			(width 0)
+			(type default)
+		)
+	)
+	(wire
+		(pts
 			(xy 215.9 31.75) (xy 227.33 31.75)
 		)
@@
 	(wire
 		(pts
-			(xy 269.24 121.92) (xy 274.32 121.92)
+			(xy 269.24 124.46) (xy 274.32 124.46)
 		)
 		(stroke
@@
 	(symbol
 		(lib_id "Device:R_Small")
+		(at 269.24 116.84 270)
+		(unit 1)
+		(body_style 1)
+		(exclude_from_sim no)
+		(in_bom yes)
+		(on_board yes)
+		(in_pos_files yes)
+		(dnp no)
+		(property "Reference" "R31"
+			(at 269.24 120.396 90)
+			(show_name no)
+			(do_not_autoplace no)
+			(effects
+				(font
+					(size 1.016 1.016)
+				)
+			)
+		)
+		(property "Value" "1M"
+			(at 269.24 118.872 90)
+			(show_name no)
+			(do_not_autoplace no)
+			(effects
+				(font
+					(size 1.27 1.27)
+				)
+			)
+		)
+		(property "Footprint" ""
+			(at 269.24 116.84 0)
+			(hide yes)
+			(show_name no)
+			(do_not_autoplace no)
+			(effects
+				(font
+					(size 1.27 1.27)
+				)
+			)
+		)
+		(property "Datasheet" ""
+			(at 269.24 116.84 0)
+			(hide yes)
+			(show_name no)
+			(do_not_autoplace no)
+			(effects
+				(font
+					(size 1.27 1.27)
+				)
+			)
+		)
+		(property "Description" "Resistor, small symbol"
+			(at 269.24 116.84 0)
+			(hide yes)
+			(show_name no)
+			(do_not_autoplace no)
+			(effects
+				(font
+					(size 1.27 1.27)
+				)
+			)
+		)
+		(pin "1"
+		)
+		(pin "2"
+		)
+		(instances
+			(project "USB-C_3.2gen1"
+				(path "/d3213dd5-4179-4001-95f6-ec74c0d8f8ed/f5cb6dae-f4e5-4740-8d04-47b64833c5c2"
+					(reference "R31")
+					(unit 1)
+				)
+			)
+		)
+	)
+	(symbol
+		(lib_id "Device:R_Small")
 		(at 83.82 107.95 90)
 		(unit 1)
@@
 	(symbol
 		(lib_id "Device:C_Small")
-		(at 264.16 118.11 0)
+		(at 264.16 120.65 0)
 		(unit 1)
 		(body_style 1)
@@
 		(dnp no)
 		(property "Reference" "C48"
-			(at 257.302 117.602 0)
+			(at 257.302 120.142 0)
 			(show_name no)
 			(do_not_autoplace no)
@@
 		)
 		(property "Value" "18pF"
-			(at 257.302 120.142 0)
+			(at 257.302 122.682 0)
 			(show_name no)
 			(do_not_autoplace no)
@@
 		)
 		(property "Footprint" ""
-			(at 264.16 118.11 0)
+			(at 264.16 120.65 0)
 			(hide yes)
 			(show_name no)
@@
 		)
 		(property "Datasheet" ""
-			(at 264.16 118.11 0)
+			(at 264.16 120.65 0)
 			(hide yes)
 			(show_name no)
@@
 		)
 		(property "Description" "Unpolarized capacitor, small symbol"
-			(at 264.16 118.11 0)
+			(at 264.16 120.65 0)
 			(hide yes)
 			(show_name no)
@@
 	(symbol
 		(lib_id "Device:C_Small")
-		(at 274.32 118.11 0)
+		(at 274.32 120.65 0)
 		(mirror y)
 		(unit 1)
@@
 		(dnp no)
 		(property "Reference" "C49"
-			(at 281.178 117.602 0)
+			(at 281.178 120.142 0)
 			(show_name no)
 			(do_not_autoplace no)
@@
 		)
 		(property "Value" "18pF"
-			(at 281.178 120.142 0)
+			(at 281.178 122.682 0)
 			(show_name no)
 			(do_not_autoplace no)
@@
 		)
 		(property "Footprint" ""
-			(at 274.32 118.11 0)
+			(at 274.32 120.65 0)
 			(hide yes)
 			(show_name no)
@@
 		)
 		(property "Datasheet" ""
-			(at 274.32 118.11 0)
+			(at 274.32 120.65 0)
 			(hide yes)
 			(show_name no)
@@
 		)
 		(property "Description" "Unpolarized capacitor, small symbol"
-			(at 274.32 118.11 0)
+			(at 274.32 120.65 0)
 			(hide yes)
 			(show_name no)
@@
 	(symbol
 		(lib_id "power:GND")
-		(at 269.24 123.19 0)
+		(at 269.24 125.73 0)
 		(mirror y)
 		(unit 1)
@@
 		(dnp no)
 		(property "Reference" "#PWR049"
-			(at 269.24 129.54 0)
+			(at 269.24 132.08 0)
 			(hide yes)
 			(show_name no)
@@
 		)
 		(property "Value" "GND"
-			(at 265.176 124.714 0)
+			(at 265.176 127.254 0)
 			(show_name no)
 			(do_not_autoplace no)
@@
 		)
 		(property "Footprint" ""
-			(at 269.24 123.19 0)
+			(at 269.24 125.73 0)
 			(hide yes)
 			(show_name no)
@@
 		)
 		(property "Datasheet" ""
-			(at 269.24 123.19 0)
+			(at 269.24 125.73 0)
 			(hide yes)
 			(show_name no)
@@
 		)
 		(property "Description" "Power symbol creates a global label with name \"GND\" , ground"
-			(at 269.24 123.19 0)
+			(at 269.24 125.73 0)
 			(hide yes)
 			(show_name no)

Commit message: Add files via upload
Parts:
- C2, C23, C24, C3, C4, C42, C43, C44, C45, C46, C47, C48, C49, C5, C50, C51, C54, C55, C56, C57, C58, C59, C60, C61, C62, C63, C64, C65, C66, C67: footprint (none) -> Capacitor_SMD:C_0603_1608Metric
- C68: footprint (none) -> Capacitor_SMD:C_1206_3216Metric
- F1: footprint (none) -> Fuse:Fuse_1206_3216Metric
- J4: footprint (none) -> Connector_USB:USB3_A_Plug_Wuerth_692112030100_Horizontal
- R14, R20, R21, R22, R23, R31: footprint (none) -> Resistor_SMD:R_0603_1608Metric
- U4: footprint QFN76_RTK -> Package_DFN_QFN:QFN-76-1EP_9x9mm_P0.4mm_EP5.81x6.31mm_ThermalVias
- Y1: footprint (none) -> Crystal:Crystal_SMD_3225-4Pin_3.2x2.5mm
Changed lines of the file:
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@@
 			)
 		)
-		(property "Footprint" ""
+		(property "Footprint" "Capacitor_SMD:C_0603_1608Metric"
 			(at 163.83 156.21 0)
 			(hide yes)
@@
 			)
 		)
-		(property "Footprint" ""
+		(property "Footprint" "Capacitor_SMD:C_0603_1608Metric"
 			(at 208.28 134.62 0)
 			(hide yes)
@@
 			)
 		)
-		(property "Footprint" ""
+		(property "Footprint" "Capacitor_SMD:C_0603_1608Metric"
 			(at 146.05 90.17 0)
 			(hide yes)
@@
 			)
 		)
-		(property "Footprint" ""
+		(property "Footprint" "Crystal:Crystal_SMD_3225-4Pin_3.2x2.5mm"
 			(at 269.24 113.03 0)
 			(hide yes)
@@
 			)
 		)
-		(property "Footprint" ""
+		(property "Footprint" "Capacitor_SMD:C_0603_1608Metric"
 			(at 139.7 57.15 0)
 			(hide yes)
@@
 			)
 		)
-		(property "Footprint" ""
+		(property "Footprint" "Capacitor_SMD:C_0603_1608Metric"
 			(at 240.03 67.31 0)
 			(hide yes)
@@
 			)
 		)
-		(property "Footprint" ""
+		(property "Footprint" "Resistor_SMD:R_0603_1608Metric"
 			(at 269.24 116.84 0)
 			(hide yes)
@@
 			)
 		)
-		(property "Footprint" ""
+		(property "Footprint" "Resistor_SMD:R_0603_1608Metric"
 			(at 83.82 107.95 0)
 			(hide yes)
@@
 			)
 		)
-		(property "Footprint" ""
+		(property "Footprint" "Capacitor_SMD:C_0603_1608Metric"
 			(at 139.7 87.63 0)
 			(hide yes)
@@
 			)
 		)
-		(property "Footprint" ""
+		(property "Footprint" "Capacitor_SMD:C_0603_1608Metric"
 			(at 251.46 96.52 0)
 			(hide yes)
@@
 			)
 		)
-		(property "Footprint" ""
+		(property "Footprint" "Capacitor_SMD:C_0603_1608Metric"
 			(at 264.16 120.65 0)
 			(hide yes)
@@
 			)
 		)
-		(property "Footprint" ""
+		(property "Footprint" "Capacitor_SMD:C_0603_1608Metric"
 			(at 242.57 99.06 0)
 			(hide yes)
@@
 			)
 		)
-		(property "Footprint" ""
+		(property "Footprint" "Capacitor_SMD:C_0603_1608Metric"
 			(at 251.46 45.72 0)
 			(hide yes)
@@
 			)
 		)
-		(property "Footprint" ""
+		(property "Footprint" "Capacitor_SMD:C_0603_1608Metric"
 			(at 121.92 31.75 0)
 			(hide yes)
@@
 			)
 		)
-		(property "Footprint" ""
+		(property "Footprint" "Capacitor_SMD:C_0603_1608Metric"
 			(at 274.32 120.65 0)
 			(hide yes)
@@
 			)
 		)
-		(property "Footprint" ""
+		(property "Footprint" "Capacitor_SMD:C_0603_1608Metric"
 			(at 261.62 60.96 0)
 			(hide yes)
@@
 			)
 		)
-		(property "Footprint" ""
+		(property "Footprint" "Resistor_SMD:R_0603_1608Metric"
 			(at 90.17 110.49 0)
 			(hide yes)
@@
 			)
 		)
-		(property "Footprint" ""
+		(property "Footprint" "Capacitor_SMD:C_0603_1608Metric"
 			(at 248.92 134.62 0)
 			(hide yes)
@@
 			)
 		)
-		(property "Footprint" ""
+		(property "Footprint" "Capacitor_SMD:C_1206_3216Metric"
 			(at 99.06 106.68 0)
 			(hide yes)
@@
 			)
 		)
-		(property "Footprint" "QFN76_RTK"
+		(property "Footprint" "Package_DFN_QFN:QFN-76-1EP_9x9mm_P0.4mm_EP5.81x6.31mm_ThermalVias"
 			(at 149.86 24.13 0)
 			(hide yes)
@@
 			)
 		)
-		(property "Footprint" ""
+		(property "Footprint" "Capacitor_SMD:C_0603_1608Metric"
 			(at 223.52 54.61 0)
 			(hide yes)
@@
 			)
 		)
-		(property "Footprint" ""
+		(property "Footprint" "Capacitor_SMD:C_0603_1608Metric"
 			(at 87.63 138.43 0)
 			(hide yes)
@@
 			)
 		)
-		(property "Footprint" ""
+		(property "Footprint" "Capacitor_SMD:C_0603_1608Metric"
 			(at 146.05 59.69 0)
 			(hide yes)
@@
 			)
 		)
-		(property "Footprint" ""
+		(property "Footprint" "Capacitor_SMD:C_0603_1608Metric"
 			(at 139.7 41.91 0)
 			(hide yes)
@@
 			)
 		)
-		(property "Footprint" ""
+		(property "Footprint" "Capacitor_SMD:C_0603_1608Metric"
 			(at 157.48 158.75 0)
 			(hide yes)
@@
 			)
 		)
-		(property "Footprint" ""
+		(property "Footprint" "Capacitor_SMD:C_0603_1608Metric"
 			(at 113.03 43.18 0)
 			(hide yes)
@@
 			)
 		)
-		(property "Footprint" ""
+		(property "Footprint" "Capacitor_SMD:C_0603_1608Metric"
 			(at 111.76 88.9 0)
 			(hide yes)
@@
 			)
 		)
-		(property "Footprint" ""
+		(property "Footprint" "Capacitor_SMD:C_0603_1608Metric"
 			(at 233.68 69.85 0)
 			(hide yes)
@@
 			)
 		)
-		(property "Footprint" ""
+		(property "Footprint" "Capacitor_SMD:C_0603_1608Metric"
 			(at 121.92 104.14 0)
 			(hide yes)
@@
 			)
 		)
-		(property "Footprint" ""
+		(property "Footprint" "Capacitor_SMD:C_0603_1608Metric"
 			(at 113.03 58.42 0)
 			(hide yes)
@@
 			)
 		)
-		(property "Footprint" ""
+		(property "Footprint" "Resistor_SMD:R_0603_1608Metric"
 			(at 243.84 49.53 0)
 			(hide yes)
@@
 			)
 		)
-		(property "Footprint" ""
+		(property "Footprint" "Capacitor_SMD:C_0603_1608Metric"
 			(at 246.38 83.82 0)
 			(hide yes)
@@
 			)
 		)
-		(property "Footprint" ""
+		(property "Footprint" "Resistor_SMD:R_0603_1608Metric"
 			(at 137.16 24.13 0)
 			(hide yes)
@@
 			)
 		)
-		(property "Footprint" ""
+		(property "Footprint" "Capacitor_SMD:C_0603_1608Metric"
 			(at 247.65 74.93 0)
 			(hide yes)
@@
 			)
 		)
-		(property "Footprint" ""
+		(property "Footprint" "Fuse:Fuse_1206_3216Metric"
 			(at 157.48 134.62 0)
 			(hide yes)
@@
 			)
 		)
-		(property "Footprint" ""
+		(property "Footprint" "Capacitor_SMD:C_0603_1608Metric"
 			(at 121.92 73.66 0)
 			(hide yes)
@@
 			)
 		)
-		(property "Footprint" ""
+		(property "Footprint" "Resistor_SMD:R_0603_1608Metric"
 			(at 123.19 46.99 0)
 			(hide yes)
@@
 			)
 		)
-		(property "Footprint" ""
+		(property "Footprint" "Capacitor_SMD:C_0603_1608Metric"
 			(at 93.98 135.89 0)
 			(hide yes)
@@
 			)
 		)
-		(property "Footprint" ""
+		(property "Footprint" "Capacitor_SMD:C_0603_1608Metric"
 			(at 229.87 52.07 0)
 			(hide yes)
@@
 			)
 		)
-		(property "Footprint" ""
+		(property "Footprint" "Capacitor_SMD:C_0603_1608Metric"
 			(at 146.05 44.45 0)
 			(hide yes)
@@
 			)
 		)
-		(property "Footprint" ""
+		(property "Footprint" "Connector_USB:USB3_A_Plug_Wuerth_692112030100_Horizontal"
 			(at 138.43 143.51 0)
 			(hide yes)

Commit message: Add files via upload
Other:
- moved on the sheet: C2, C23, C24, C3, C4, C42, C43, C44, C45, C46, C47, C48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

Commit message: Add files via upload
Parts:
- renumbered C66 to C36, C67 to C37, C68 to C38, C43 to C39, C23 to C40, C24 to C41, C3 to C42, C42 to C43, C57 to C45, C58 to C46, C60 to C47, C56 to C48, C59 to C49, C61 to C50, C64 to C51, C65 to C52, C63 to C53, C50 to C56, C51 to C57, C5 to C58, C2 to C59, C47 to C60, C62 to C61, C45 to C62, C4 to C63, C46 to C64, C48 to C65, C49 to C66, J5 to J3, R20 to R24, R14 to R25, R21 to R26, R31 to R27, U19 to U13, U18 to U14, U4 to U15, U17 to U16, U16 to U17
