File: USB-C_3.2gen1.kicad_pcb (KiCad board)
At the start: 2 copper layers, 168 parts, among them J1 USB_C_Master, J2 DP_Source, J3 USB_C_Slave, J4 USB3_A, J5 USB_C_Receptacle, J6 RJ45_JK0654219, J7 112L-TDA0, J8 ST50S017VCAR1800, U1 AP63200WU, U10 TPD4S311YBFR, U11 TPD2S300YFFR, U12 W25Q16JVSSIQ, U13 TPS65988DHRSHR, U14 AP63200WU, U15 TLV70012_SOT23-5, U16 USBLC6-2SC6, U17 USBLC6-2SC6, U18 TPD4E05U06DQA, U19 TPD4E05U06DQA, U2 TPD4E05U06DQA, U20 RTL8153B-VB-CG, U3 TPD4E05U06DQA, U4 RTS5411-GRT, U5 TUSB564IRNQR, U6 GL3224-ONY, U8 TPD4E05U06DQA, U9 USBLC6-2SC6, Y1 24MHz, Y2 25MHz, Y3 12MHz

Commit message: Add files via upload
Parts:
- removed C98, C99: 4,7uF, Capacitor_SMD:C_1206_3216Metric
- removed U20: RTL8153B-VB-CG, RTL8153B-VB-CG:QFN40P500X500X90-41N
- added C11: 22uF, Capacitor_SMD:C_1206_3216Metric, F.Cu at (28.9, 29.5)
- added C31: 100nF, Capacitor_SMD:C_0603_1608Metric, F.Cu at (203.5, 101.9)
- added U7: TPD4S311YBFR, Package_BGA:Texas_DSBGA-16_2.39x2.39mm_Layout4x4_P0.5mm, F.Cu at (200.2, 118.5)
- C1, C27, C33, C68: value 10uF -> 100nF; footprint Capacitor_SMD:C_1206_3216Metric -> Capacitor_SMD:C_0603_1608Metric
- C10, C12, C13: value 100nF -> 22uF; footprint Capacitor_SMD:C_0603_1608Metric -> Capacitor_SMD:C_1206_3216Metric
- C14, C15, C59, C6: value 100nF -> 1uF
- C16, C17, C21: value 100nF -> 2,2uF
- C18, C2, C52, C53: value 1uF -> 100nF
- C20, C3, C4, C82: value 100nF -> 10uF; footprint Capacitor_SMD:C_0603_1608Metric -> Capacitor_SMD:C_1206_3216Metric
- C22: value 1uF -> 2,2uF
- C23, C67: value 100nF -> 10nF
- C25: value 2,2uF -> 1uF
- C26, C29, C30: value 2,2uF -> 100nF
- C35, C36, C40, C41: value 22uF -> 100nF; footprint Capacitor_SMD:C_1206_3216Metric -> Capacitor_SMD:C_0603_1608Metric
- C48, C49, C71, C72: value 18pF -> 100nF
- C65, C66, C69, C70: value 100nF -> 18pF
- C7: value 10nF -> 10uF; footprint Capacitor_SMD:C_0603_1608Metric -> Capacitor_SMD:C_1206_3216Metric
- C74, C89, C91: value 100nF -> 4,7uF; footprint Capacitor_SMD:C_0603_1608Metric -> Capacitor_SMD:C_1206_3216Metric
- C79, C97: value 4,7uF -> 100nF; footprint Capacitor_SMD:C_1206_3216Metric -> Capacitor_SMD:C_0603_1608Metric
- C81: value 10nF -> 100nF
- C92, C94: value 10uF -> 4,7uF
- C96: value 4,7uF -> 10uF
- J1: value USB_C_Master -> USB_C_Slave
- J2: value DP_Source -> USB_C_Master; footprint DPF20102741TR:AMPHENOL_DPF20102741TR -> Connector_USB:USB_C_Receptacle_Molex_105450-0101
- J3: value USB_C_Slave -> USB_C_Receptacle
- J5: value USB_C_Receptacle -> DP_Source; footprint Connector_USB:USB_C_Receptacle_Molex_105450-0101 -> DPF20102741TR:AMPHENOL_DPF20102741TR
- J8: value ST50S017VCAR1800 -> 112L-TDA0; footprint ST50S017VCAR1800:ST50S017VCAR1800_JAE -> 112L-TDA0:CONN_112L-TDA0_ATT
- R1, R13, R15, R20, R21, R9: value 10K -> 100K
- R10: value 52K3 -> 10K
- R11: value 10K -> 4K7
- R12: value 100K -> 4K7
- R14: value 12K1 -> 1M
- R16, R17: value 100K -> 2M
- R18, R19, R6: value 100K -> 10K
- R2: value 2M -> 100K
- R24: value 2K49 -> 10K
- R25: value 330R -> 12K1
- R26: value 330R -> 10K
- R28: value 10K, 1% -> 1M
- R29: value 330R -> 2K49
- R3: value 1M -> 52K3
- R30: value 10K -> 330R
- R31: value 1M -> 330R
- R32: value 4K7 -> 10K, 1%
- R33: value 4K7 -> 330R
- R4: value 2M -> 10K
- R5: value 100K -> 31K6
- R8: value 31K6 -> 10K
- U10: value TPD4S311YBFR -> USBLC6-2SC6; footprint Package_BGA:Texas_YFP0020_DSBGA-20_1.588x1.988mm_Layout4x5_P0.4mm -> Package_TO_SOT_SMD:SOT-23-6
- U11: value TPD2S300YFFR -> TPD4E05U06DQA; footprint Package_BGA:Texas_DSBGA-28_1.9x3mm_Layout4x7_P0.4mm -> Package_SON:USON-10_2.5x1.0mm_P0.5mm
- U12: value W25Q16JVSSIQ -> TUSB564IRNQR; footprint W25Q16JVSSIQ:SOIC127P790X216-8N -> Package_DFN_QFN:Texas_RNQ0040A_WQFN-40-1EP_6x4mm_P0.4mm_EP4.7x2.7mm_ThermalVias
- U13: value TPS65988DHRSHR -> TPD4E05U06DQA; footprint TPS65988DHRSHR:IC_TPS65987DDHRSHR -> Package_SON:USON-10_2.5x1.0mm_P0.5mm
- U14: value AP63200WU -> TPD4E05U06DQA; footprint Package_TO_SOT_SMD:TSOT-23-6 -> Package_SON:USON-10_2.5x1.0mm_P0.5mm
- U15: value TLV70012_SOT23-5 -> RTS5411-GRT; footprint Package_TO_SOT_SMD:SOT-23-5 -> Package_DFN_QFN:QFN-76-1EP_9x9mm_P0.4mm_EP5.81x6.31mm_ThermalVias
- U18: value TPD4E05U06DQA -> RTL8153B-VB-CG; footprint Package_SON:USON-10_2.5x1.0mm_P0.5mm -> RTL8153B-VB-CG:QFN40P500X500X90-41N
- U19: value TPD4E05U06DQA -> GL3224-ONY; footprint Package_SON:USON-10_2.5x1.0mm_P0.5mm -> Package_DFN_QFN:QFN-48-1EP_7x7mm_P0.5mm_EP5.15x5.15mm
- U2: value TPD4E05U06DQA -> AP63200WU; footprint Package_SON:USON-10_2.5x1.0mm_P0.5mm -> Package_TO_SOT_SMD:TSOT-23-6
- U3: value TPD4E05U06DQA -> TPD2S300YFFR; footprint Package_SON:USON-10_2.5x1.0mm_P0.5mm -> Package_BGA:Texas_DSBGA-9_1.4715x1.4715mm_Layout3x3_P0.5mm
- U4: value RTS5411-GRT -> TLV70012_SOT23-5; footprint Package_DFN_QFN:QFN-76-1EP_9x9mm_P0.4mm_EP5.81x6.31mm_ThermalVias -> Package_TO_SOT_SMD:SOT-23-5
- U5: value TUSB564IRNQR -> TPS65988DHRSHR; footprint Package_DFN_QFN:Texas_RNQ0040A_WQFN-40-1EP_6x4mm_P0.4mm_EP4.7x2.7mm_ThermalVias -> TPS65988DHRSHR:IC_TPS65987DDHRSHR
- U6: value GL3224-ONY -> W25Q16JVSSIQ; footprint Package_DFN_QFN:QFN-48-1EP_7x7mm_P0.5mm_EP5.15x5.15mm -> W25Q16JVSSIQ:SOIC127P790X216-8N
- U9: value USBLC6-2SC6 -> TPD4E05U06DQA; footprint Package_TO_SOT_SMD:SOT-23-6 -> Package_SON:USON-10_2.5x1.0mm_P0.5mm
- moved U4 174.3 mm to (44.9, 24.8)
- moved R6 171.7 mm to (19.2, 22.2)
- moved R5 169.9 mm to (17.9, 24.5), turned to 90 degrees
- moved U2 167.2 mm to (20.9, 24.8)
- moved U6 164.7 mm to (45.6, 42.7)
- moved R2 164.2 mm to (18.0, 27.6), turned to 90 degrees
- moved L2 160.0 mm to (27.5, 24.9)
- moved C9 159.8 mm to (22.2, 22.2), turned to 180 degrees
- moved R1 157.5 mm to (18.4, 48.4), turned to 90 degrees
- moved R4 157.4 mm to (19.9, 43.0)
- moved R3 156.5 mm to (18.4, 45.3), turned to 90 degrees
- moved C13 153.1 mm to (28.9, 31.9), turned to 180 degrees
- moved D1 151.7 mm to (30.9, 69.1)
- moved J1 151.5 mm to (21.6, 71.6)
- moved L1 150.2 mm to (28.3, 45.6)
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Connections:
- C1 pad 1: /POWER/VBUS1 -> SYS_PWR
- C10 pad 1: /USB-C MUX/3V3 -> 5V
- C12 pad 1: Net-(U5-SSRXN) -> 5V
- C12 pad 2: /USB-C MUX/HUB_SSTX- -> GND
- C13 pad 1: Net-(U5-SSRXP) -> 3V3
- C13 pad 2: /USB-C MUX/HUB_SSTX+ -> GND
- C14 pad 1: Net-(U5-DP0P) -> 3V3
- C14 pad 2: /USB-C MUX/DP_ML0+ -> GND
- C15 pad 1: Net-(U5-DP0N) -> 1V2
- C15 pad 2: /USB-C MUX/DP_ML0- -> GND
- C16 pad 1: Net-(U5-DP1P) -> LDO_3V3
- C16 pad 2: /USB-C MUX/DP_ML1+ -> GND
- C17 pad 1: Net-(U5-DP1N) -> Net-(U5-LDO_1V8)
- C17 pad 2: /USB-C MUX/DP_ML1- -> GND
- C18 pad 1: GND -> LDO_3V3
- C18 pad 2: /USB-C MUX/3V3 -> GND
- C19 pad 1: Net-(U10-VBIAS) -> 3V3
- C2 pad 1: GND -> SYS_PWR
- C2 pad 2: Net-(U4-V33_OUT) -> GND
- C20 pad 1: GND -> 3V3
- C20 pad 2: /USB-C MUX/5V -> GND
- C21 pad 1: GND -> Net-(U5-PP2_CABLE)
- C21 pad 2: /POWER/5V -> GND
- C22 pad 1: /POWER/3V3 -> Net-(U5-PP1_CABLE)
- C23 pad 2: /USB HUB/1V2 -> Net-(J2-SHIELD)
- C24 pad 1: GND -> Net-(U7-VBIAS)
- C24 pad 2: /USB HUB/1V2 -> GND
- C25 pad 1: Net-(U13-PP1_CABLE) -> GND
- C25 pad 2: GND -> 3V3
- C26 pad 1: Net-(U13-PP2_CABLE) -> 3V3
- C27 pad 1: /POWER/3V3 -> Net-(C27-Pad1)
- C28 pad 1: /POWER/3V3 -> Net-(C28-Pad1)
- C29 pad 1: /POWER/LDO_3V3 -> GND
- C29 pad 2: GND -> 5V
- C3 pad 1: /USB HUB/1V2 -> SYS_PWR
- C30 pad 1: Net-(U13-LDO_1V8) -> Net-(U12-DP0P)
- C30 pad 2: GND -> DP_ML0+
- C32 pad 1: /POWER/SYS_PWR -> Net-(U12-SSRXN)
- C32 pad 2: GND -> HUB_SSTX-
- C33 pad 1: /POWER/SYS_PWR -> Net-(U12-SSRXP)
- C33 pad 2: GND -> HUB_SSTX+
- C34 pad 1: Net-(U1-SW) -> Net-(U12-DP0N)
- C34 pad 2: Net-(U1-BST) -> DP_ML0-
- C35 pad 1: /POWER/3V3 -> Net-(U12-DP1N)
- C35 pad 2: GND -> DP_ML1-
- C36 pad 1: /POWER/3V3 -> /USB HUB/USBC_SSTX+
- C36 pad 2: GND -> Net-(J3-TX1+)
- C37 pad 1: /POWER/SYS_PWR -> /USB HUB/USBC_SSTX-
- C37 pad 2: GND -> Net-(J3-TX1-)
- C38 pad 1: /POWER/SYS_PWR -> 5V
- C39 pad 1: Net-(U14-SW) -> GND
- C39 pad 2: Net-(U14-BST) -> 1V2
- C4 pad 1: /USB HUB/1V2 -> SYS_PWR
- C40 pad 1: /POWER/5V -> GND
- C40 pad 2: GND -> 1V2
- C41 pad 1: /POWER/5V -> GND
- C41 pad 2: GND -> 1V2
- C42 pad 1: GND -> 1V2
- C42 pad 2: /USB HUB/1V2 -> GND
- C43 pad 2: /USB HUB/1V2 -> 1V2
- C44 pad 2: /USB HUB/1V2 -> 1V2
- C45 pad 1: GND -> SD_SSRX+
- C45 pad 2: /USB HUB/1V2 -> Net-(U15-DSP2_SSTX+)
- C46 pad 1: GND -> /USB HUB/USBA_SSRX+
- C46 pad 2: /USB HUB/1V2 -> Net-(U15-DSP3_SSTX+)
- C47 pad 1: GND -> /USB HUB/USBC_SSRX+
- C47 pad 2: /USB HUB/1V2 -> Net-(U15-DSP4_SSTX+)
- C48 pad 1: /USB HUB/XTL0 -> SD_SSRX-
- C48 pad 2: GND -> Net-(U15-DSP2_SSTX-)
- C49 pad 1: /USB HUB/XTLI -> /USB HUB/USBA_SSRX-
- C49 pad 2: GND -> Net-(U15-DSP3_SSTX-)
- C5 pad 1: /USB HUB/1V2 -> GND
- C5 pad 2: GND -> 5V
- C50 pad 1: /USB HUB/HUB_SSRX- -> /USB HUB/USBC_SSRX-
- C50 pad 2: Net-(U4-USP_SSTX-) -> Net-(U15-DSP4_SSTX-)
- C51 pad 1: /USB HUB/HUB_SSRX+ -> /USB HUB/USBA_SSTX+
- C51 pad 2: Net-(U4-USP_SSTX+) -> Net-(J4-SSTX+)
- C52 pad 1: /POWER/3V3 -> /USB HUB/USBA_SSTX-
- C52 pad 2: GND -> Net-(J4-SSTX-)
- C53 pad 1: /POWER/1V2 -> GND
- C53 pad 2: GND -> 5V
- C54 pad 1: /USB HUB/LAN_SSRX+ -> LAN_SSRX+
- C54 pad 2: Net-(U4-DSP1_SSTX+) -> Net-(U15-DSP1_SSTX+)
- C55 pad 1: /USB HUB/LAN_SSRX- -> LAN_SSRX-
- C55 pad 2: Net-(U4-DSP1_SSTX-) -> Net-(U15-DSP1_SSTX-)
- C56 pad 1: /USB HUB/SD_SSRX- -> HUB_SSRX-
- C56 pad 2: Net-(U4-DSP2_SSTX-) -> Net-(U15-USP_SSTX-)
- C57 pad 1: /USB HUB/SD_SSRX+ -> HUB_SSRX+
- C57 pad 2: Net-(U4-DSP2_SSTX+) -> Net-(U15-USP_SSTX+)
- C58 pad 1: /USB HUB/USBA_SSRX+ -> 1V2
- C58 pad 2: Net-(U4-DSP3_SSTX+) -> GND
- C59 pad 1: /USB HUB/USBA_SSRX- -> GND
- C59 pad 2: Net-(U4-DSP3_SSTX-) -> Net-(U15-V33_OUT)
- C6 pad 1: /POWER/LDO_3V3 -> 3V3
- C60 pad 1: /USB HUB/USBC_SSRX+ -> GND
- C60 pad 2: Net-(U4-DSP4_SSTX+) -> 1V2
- C61 pad 1: /USB HUB/USBC_SSRX- -> GND
- C61 pad 2: Net-(U4-DSP4_SSTX-) -> 5V
- C62 pad 2: /USB HUB/5V -> 1V2
- C63 pad 1: GND -> 1V2
- C63 pad 2: /USB HUB/5V -> GND
- C64 pad 1: /USB HUB/USBA_SSTX+ -> GND
- C64 pad 2: Net-(J4-SSTX+) -> 1V2
- C65 pad 1: /USB HUB/USBA_SSTX- -> XTL0
- C65 pad 2: Net-(J4-SSTX-) -> GND
- C66 pad 1: /USB HUB/USBC_SSTX+ -> XTLI
- C66 pad 2: Net-(J5-TX1+) -> GND
- C67 pad 1: /USB HUB/USBC_SSTX- -> Net-(C67-Pad1)
- C67 pad 2: Net-(J5-TX1-) -> GND
- C68 pad 1: /USB HUB/5V -> Net-(J6-MXCT1)
- C69 pad 1: /ETHERNET/LAN_SSTX- -> /ETHERNET/CKXTAL1
- C69 pad 2: Net-(U20-U3SSTXN) -> GND
- C7 pad 1: GND -> VBUS1
- C7 pad 2: Net-(J1-SHIELD) -> GND
- C70 pad 1: /ETHERNET/LAN_SSTX+ -> /ETHERNET/CKXTAL2
- C70 pad 2: Net-(U20-U3SSTXP) -> GND
- C71 pad 1: /ETHERNET/CKXTAL1 -> LAN_SSTX-
- C71 pad 2: GND -> Net-(U18-U3SSTXN)
- C72 pad 1: /ETHERNET/CKXTAL2 -> GND
- C72 pad 2: GND -> AVDD10
- C74 pad 1: GND -> AVDD10
- C74 pad 2: AVDD10 -> GND
- C75 pad 1: GND -> LAN_SSTX+
- C75 pad 2: AVDD10 -> Net-(U18-U3SSTXP)
- C78 pad 1: AVDD10 -> GND
- C78 pad 2: GND -> AVDD10
- C8 pad 1: Net-(C8-Pad1) -> Net-(U1-SW)
- C8 pad 2: GND -> Net-(U1-BST)
- C80 pad 1: Net-(J6-MXCT1) -> 3V3
- C81 pad 1: Net-(C81-Pad1) -> 3V3
- C82 pad 1: AVDD33 -> /SD/VDD(2)
- C83 pad 1: AVDD33 -> /SD/VDD(2)
- C86 pad 1: /SD/SD_SSTX+ -> SD_SSTX-
- C86 pad 2: Net-(U6-TXP) -> Net-(U19-TXN)
- C87 pad 1: /SD/SD_SSTX- -> SD_SSTX+
- C87 pad 2: Net-(U6-TXN) -> Net-(U19-TXP)
- C88 pad 1: /SD/3V3 -> Net-(U19-AVDD12)
- C89 pad 1: /SD/3V3 -> Net-(U19-AVDD12)
- C9 pad 1: Net-(C9-Pad1) -> Net-(U2-SW)
- C9 pad 2: GND -> Net-(U2-BST)
- C90 pad 1: Net-(U6-DVDD12) -> Net-(U19-DVDD12)
- C91 pad 1: Net-(U6-AVDD12) -> Net-(U19-DVDD12)
- C92 pad 1: /SD/VDD(2) -> 3V3
- C93 pad 1: /SD/VDD(2) -> 3V3
- C94 pad 1: /SD/VDD -> 3V3
- C95 pad 1: /SD/VDD -> 3V3
- C96 pad 1: /SD/3V3 -> /SD/VDD
- C97 pad 1: /SD/3V3 -> /SD/VDD
- D1 pad 1: /USB-C MUX/VBUS2 -> VBUS1
- D2 pad 1: /POWER/VBUS1 -> VBUS2
- F1 pad 2: /USB HUB/5V -> 5V
- J1 pad A10: /USB-C MUX/RX2- -> unconnected-(J1-RX2--PadA10)
- J1 pad A11: /USB-C MUX/RX2+ -> unconnected-(J1-RX2+-PadA11)
- J1 pad A2: /USB-C MUX/TX1+ -> unconnected-(J1-TX1+-PadA2)
- J1 pad A3: /USB-C MUX/TX1- -> unconnected-(J1-TX1--PadA3)
- J1 pad A4: /USB-C MUX/VBUS2 -> VBUS1
- J1 pad A5: /USB-C MUX/C_CC1 -> /POWER/C_CC1(2)
- J1 pad A6: /USB-C MUX/USB2*_D+ -> unconnected-(J1-D+-PadA6)
- J1 pad A7: /USB-C MUX/USB2*_D- -> unconnected-(J1-D--PadA7)
- J1 pad A8: /USB-C MUX/SBU*1 -> unconnected-(J1-SBU1-PadA8)
- J1 pad A9: /USB-C MUX/VBUS2 -> VBUS1
- J1 pad B10: /USB-C MUX/RX1- -> unconnected-(J1-RX1--PadB10)
- J1 pad B11: /USB-C MUX/RX1+ -> unconnected-(J1-RX1+-PadB11)
- J1 pad B2: /USB-C MUX/TX2+ -> unconnected-(J1-TX2+-PadB2)
- J1 pad B3: /USB-C MUX/TX2- -> unconnected-(J1-TX2--PadB3)
- J1 pad B4: /USB-C MUX/VBUS2 -> VBUS1
- J1 pad B5: /USB-C MUX/C_CC2 -> /POWER/C_CC2(2)
- J1 pad B6: /USB-C MUX/USB2*_D+ -> unconnected-(J1-D+-PadB6)
- J1 pad B7: /USB-C MUX/USB2*_D- -> unconnected-(J1-D--PadB7)
- J1 pad B8: /USB-C MUX/SBU*2 -> unconnected-(J1-SBU2-PadB8)
- J1 pad B9: /USB-C MUX/VBUS2 -> VBUS1
- J1 pad SH: Net-(J1-SHIELD) -> GND
- J3 pad A2: unconnected-(J3-TX1+-PadA2) -> Net-(J3-TX1+)
- J3 pad A3: unconnected-(J3-TX1--PadA3) -> Net-(J3-TX1-)
- J3 pad A4: /POWER/VBUS1 -> 5V
- J3 pad A5: /POWER/C_CC1(2) -> Net-(J3-CC1)
- J3 pad A6: unconnected-(J3-D+-PadA6) -> /USB HUB/USBC_*D+
- J3 pad A7: unconnected-(J3-D--PadA7) -> /USB HUB/USBC_*D-
- J3 pad A9: /POWER/VBUS1 -> 5V
- J3 pad B10: unconnected-(J3-RX1--PadB10) -> /USB HUB/USBC_SSRX-
- J3 pad B11: unconnected-(J3-RX1+-PadB11) -> /USB HUB/USBC_SSRX+
- J3 pad B4: /POWER/VBUS1 -> 5V
- J3 pad B5: /POWER/C_CC2(2) -> Net-(J3-CC2)
- J3 pad B6: unconnected-(J3-D+-PadB6) -> /USB HUB/USBC_*D+
- J3 pad B7: unconnected-(J3-D--PadB7) -> /USB HUB/USBC_*D-
- J3 pad B9: /POWER/VBUS1 -> 5V
- J6 pad 14: AVDD33 -> 3V3
- J6 pad 16: AVDD33 -> 3V3
- J6 pad SH: Net-(C81-Pad1) -> Net-(C67-Pad1)
- J8 pad 17: /SD/SWIO -> GND
- L1 pad 2: /POWER/3V3 -> 5V
- L2 pad 1: Net-(U14-SW) -> Net-(U2-SW)
- L2 pad 2: /POWER/5V -> 3V3
- L3 pad 1: Net-(U20-REGOUT) -> Net-(U18-REGOUT)
- R1 pad 1: /USB-C MUX/3V3 -> SYS_PWR
- R1 pad 2: Net-(U5-I2C_EN) -> Net-(U1-EN)
- R10 pad 1: /POWER/5V -> Net-(U5-HRESET)
- R10 pad 2: Net-(U14-FB) -> GND
- R11 pad 1: Net-(U14-FB) -> 3V3
- R11 pad 2: GND -> I2C_SDA
- R12 pad 1: /POWER/LDO_3V3 -> 3V3
- R12 pad 2: Net-(U12-~{HOLD}/RESET(IO3)) -> I2C_SCL
- R13 pad 1: /POWER/3V3 -> LDO_3V3
- R13 pad 2: Net-(U11-FLT_N) -> Net-(U6-~{HOLD}/RESET(IO3))
- R14 pad 2: Net-(U4-RREF) -> Net-(J2-SHIELD)
- R15 pad 1: Net-(U13-HRESET) -> 3V3
- R15 pad 2: GND -> Net-(U7-FLT)
- R16 pad 1: Net-(U13-ADCIN2) -> GND
- R16 pad 2: GND -> SBU2
- R17 pad 1: Net-(U13-ADCIN1) -> GND
- R17 pad 2: GND -> SBU1
- R18 pad 1: /POWER/SYS_PWR -> 3V3
- R18 pad 2: Net-(U1-EN) -> Net-(U12-EN)
- R19 pad 1: /POWER/SYS_PWR -> 3V3
- R19 pad 2: Net-(U14-EN) -> Net-(U12-I2C_EN)
- R2 pad 1: GND -> SYS_PWR
- R2 pad 2: /USB-C MUX/SBU2 -> Net-(U2-EN)
- R20 pad 1: Net-(U4-OCP2) -> DP_AUX-
- R20 pad 2: /USB HUB/3V3 -> 3V3
- R21 pad 1: Net-(U4-OCP1) -> GND
- R21 pad 2: /USB HUB/3V3 -> DP_AUX+
- R22 pad 1: Net-(J5-CC1) -> Net-(J3-CC1)
- R22 pad 2: /USB HUB/5V -> 5V
- R23 pad 1: Net-(J5-CC2) -> Net-(J3-CC2)
- R23 pad 2: /USB HUB/5V -> 5V
- R24 pad 1: GND -> Net-(U15-OCP2)
- R24 pad 2: Net-(U20-RSET) -> 3V3
- R25 pad 1: Net-(U20-LED0/SPICSB) -> GND
- R25 pad 2: /ETHERNET/LED0 -> Net-(U15-RREF)
- R26 pad 1: Net-(U20-EESK/LED1/SPISCK) -> Net-(U15-OCP1)
- R26 pad 2: /ETHERNET/LED1 -> 3V3
- R27 pad 1: Net-(C81-Pad1) -> XTLI
- R27 pad 2: GND -> XTL0
- R28 pad 1: Net-(U6-RTERM) -> Net-(C67-Pad1)
- R29 pad 1: Net-(D3-K) -> GND
- R29 pad 2: GND -> Net-(U18-RSET)
- R3 pad 1: GND -> 5V
- R3 pad 2: Net-(J1-SHIELD) -> Net-(U1-FB)
- R30 pad 1: Net-(U6-MS2_INS/SD2_WP) -> Net-(U18-LED0/SPICSB)
- R30 pad 2: GND -> /ETHERNET/LED0
- R31 pad 1: /USB HUB/XTLI -> Net-(U18-EESK/LED1/SPISCK)
- R31 pad 2: /USB HUB/XTL0 -> /ETHERNET/LED1
- R32 pad 1: /POWER/3V3 -> Net-(U19-RTERM)
- R32 pad 2: /POWER/I2C_SDA -> GND
- R33 pad 1: /POWER/3V3 -> Net-(D3-K)
- R33 pad 2: /POWER/I2C_SCL -> GND
- R34 pad 1: /USB-C MUX/3V3 -> Net-(U19-MS2_INS/SD2_WP)
- R34 pad 2: Net-(U5-EN) -> GND
- R4 pad 1: GND -> Net-(U1-FB)
- R4 pad 2: /USB-C MUX/SBU1 -> GND
- R5 pad 1: /USB-C MUX/DP_AUX- -> 3V3
- R5 pad 2: /USB-C MUX/3V3 -> Net-(U2-FB)
- R6 pad 1: GND -> Net-(U2-FB)
- R6 pad 2: /USB-C MUX/DP_AUX+ -> GND
- R7 pad 1: /USB-C MUX/3V3 -> Net-(U5-ADCIN1)
- R7 pad 2: Net-(U10-FLT) -> GND
- R8 pad 1: /POWER/3V3 -> 3V3
- R8 pad 2: Net-(U1-FB) -> Net-(U3-FLT_N)
- R9 pad 1: Net-(U1-FB) -> Net-(U5-ADCIN2)
- U1 pad 3: /POWER/SYS_PWR -> SYS_PWR
- U12 pad 1: /POWER/~CS -> unconnected-(U12-NC-Pad1)
- U12 pad 2: /POWER/D0 -> unconnected-(U12-DPEQ1-Pad2)
- U12 pad 3: Net-(U12-~{HOLD}/RESET(IO3)) -> unconnected-(U12-SSEQ1-Pad3)
- U12 pad 4: GND -> Net-(U12-SSRXN)
- U12 pad 5: /POWER/D1 -> Net-(U12-SSRXP)
- U12 pad 6: /POWER/SPI_CLK -> Net-(C28-Pad1)
- U12 pad 7: Net-(U12-~{HOLD}/RESET(IO3)) -> HUB_SSRX-
- U12 pad 8: /POWER/LDO_3V3 -> HUB_SSRX+
- U13 pad 1: /POWER/SYS_PWR -> /USB HUB/USBC_SSRX+
- U13 pad 10: Net-(U13-ADCIN2) -> unconnected-(U13-NC-Pad10)
- U13 pad 3: /POWER/VBUS2 -> GND
- U13 pad 5: /POWER/3V3 -> /USB HUB/USBC_SSTX-
- U13 pad 6: Net-(U13-ADCIN1) -> unconnected-(U13-NC-Pad6)
- U13 pad 7: /POWER/VBUS2 -> unconnected-(U13-NC-Pad7)
- U13 pad 8: /POWER/VBUS1 -> GND
- U13 pad 9: /POWER/LDO_3V3 -> unconnected-(U13-NC-Pad9)
- U14 pad 1: Net-(U14-FB) -> /USB HUB/USBA_SSTX+
- U14 pad 2: Net-(U14-EN) -> /USB HUB/USBA_SSTX-
- U14 pad 3: /POWER/SYS_PWR -> GND
- U14 pad 4: GND -> /USB HUB/USBA_SSRX+
- U14 pad 5: Net-(U14-SW) -> /USB HUB/USBA_SSRX-
- U14 pad 6: Net-(U14-BST) -> unconnected-(U14-NC-Pad6)
- U15 pad 1: /POWER/3V3 -> Net-(U15-RREF)
- U15 pad 2: GND -> 3V3
- U15 pad 3: /POWER/3V3 -> 1V2
- U15 pad 4: unconnected-(U15-NC-Pad4) -> 3V3
- U15 pad 5: /POWER/1V2 -> SD_D+
- U16 pad 1: /USB HUB/USBA_*D- -> /USB HUB/USBC_*D+
- U16 pad 3: /USB HUB/USBA_*D+ -> /USB HUB/USBC_*D-
- U16 pad 4: /USB HUB/USBA_D+ -> /USB HUB/USBC_D-
- U16 pad 5: /USB HUB/5V -> 5V
- U16 pad 6: /USB HUB/USBA_D- -> /USB HUB/USBC_D+
- U17 pad 1: /USB HUB/USBC_*D+ -> /USB HUB/USBA_*D-
- U17 pad 3: /USB HUB/USBC_*D- -> /USB HUB/USBA_*D+
- U17 pad 4: /USB HUB/USBC_D- -> /USB HUB/USBA_D+
- U17 pad 5: /USB HUB/5V -> 5V
- U17 pad 6: /USB HUB/USBC_D+ -> /USB HUB/USBA_D-
- U18 pad 1: /USB HUB/USBA_SSTX+ -> /ETHERNET/MX1+
- U18 pad 10: unconnected-(U18-NC-Pad10) -> /ETHERNET/MX4-
- U18 pad 2: /USB HUB/USBA_SSTX- -> /ETHERNET/MX1-
- U18 pad 3: GND -> AVDD10
- U18 pad 4: /USB HUB/USBA_SSRX+ -> /ETHERNET/MX2+
- U18 pad 5: /USB HUB/USBA_SSRX- -> /ETHERNET/MX2-
- U18 pad 6: unconnected-(U18-NC-Pad6) -> /ETHERNET/MX3+
- U18 pad 7: unconnected-(U18-NC-Pad7) -> /ETHERNET/MX3-
- U18 pad 8: GND -> AVDD10
- U18 pad 9: unconnected-(U18-NC-Pad9) -> /ETHERNET/MX4+
- U19 pad 1: /USB HUB/USBC_SSRX+ -> /SD/SWIO
- U19 pad 10: unconnected-(U19-NC-Pad10) -> SD_SSRX-
- U19 pad 2: /USB HUB/USBC_SSRX- -> /SD/DSW1
- U19 pad 4: /USB HUB/USBC_SSTX+ -> SD_D-
- U19 pad 5: /USB HUB/USBC_SSTX- -> SD_D+
- U19 pad 6: unconnected-(U19-NC-Pad6) -> 3V3
- U19 pad 7: unconnected-(U19-NC-Pad7) -> Net-(U19-TXN)
- U19 pad 8: GND -> Net-(U19-TXP)
- U19 pad 9: unconnected-(U19-NC-Pad9) -> Net-(U19-AVDD12)
- U2 pad 1: /USB-C MUX/TX1+ -> Net-(U2-FB)
- U2 pad 2: /USB-C MUX/TX1- -> Net-(U2-EN)
- U2 pad 3: GND -> SYS_PWR
- U2 pad 4: /USB-C MUX/RX1+ -> GND
- U2 pad 5: /USB-C MUX/RX1- -> Net-(U2-SW)
- U2 pad 6: unconnected-(U2-NC-Pad6) -> Net-(U2-BST)
- U4 pad 1: Net-(U4-RREF) -> 3V3
- U4 pad 2: /USB HUB/3V3 -> GND
- U4 pad 3: /USB HUB/1V2 -> 3V3
- U4 pad 4: /USB HUB/3V3 -> unconnected-(U4-NC-Pad4)
- U4 pad 5: /USB HUB/SD_D+ -> 1V2
- U5 pad 1: unconnected-(U5-NC-Pad1) -> SYS_PWR
- U5 pad 10: /USB-C MUX/TX1- -> Net-(U5-ADCIN2)
- U5 pad 11: unconnected-(U5-EQ0-Pad11) -> SYS_PWR
- U5 pad 13: /USB-C MUX/RX1- -> VBUS1
- U5 pad 15: /USB-C MUX/RX2- -> VBUS1
- U5 pad 16: /USB-C MUX/RX2+ -> unconnected-(U5-GPIO0-Pad16)
- U5 pad 17: Net-(U5-I2C_EN) -> unconnected-(U5-GPIO1-Pad17)
- U5 pad 18: /USB-C MUX/TX2- -> unconnected-(U5-GPIO2-Pad18)
- U5 pad 19: /USB-C MUX/TX2+ -> VBUS1
- U5 pad 20: Net-(C9-Pad1) -> GND
- U5 pad 21: /USB-C MUX/I2C_SCL -> unconnected-(U5-I2C3_SCL(GPIO5)-Pad21)
- U5 pad 22: /USB-C MUX/I2C_SDA -> unconnected-(U5-I2C3_SDA(GPIO6)-Pad22)
- U5 pad 24: /USB-C MUX/SBU1 -> /POWER/CC1(2)
- U5 pad 25: /USB-C MUX/SBU2 -> Net-(U5-PP1_CABLE)
- U5 pad 26: /USB-C MUX/DP_AUX+ -> /POWER/CC2(2)
- U5 pad 27: /USB-C MUX/DP_AUX- -> I2C_SCL
- U5 pad 28: /USB-C MUX/3V3 -> I2C_SDA
- U5 pad 29: Net-(U5-EN) -> unconnected-(U5-~{I2C1_IRQ}-Pad29)
- U5 pad 3: unconnected-(U5-SSEQ1-Pad3) -> VBUS2
- U5 pad 32: /USB-C MUX/MUX_HPD -> unconnected-(U5-I2C2_SCL-Pad32)
- U5 pad 35: GND -> Net-(U5-LDO_1V8)
- U5 pad 36: Net-(U5-DP1N) -> /POWER/D0
- U5 pad 37: Net-(U5-DP1P) -> /POWER/D1
- U5 pad 38: GND -> /POWER/SPI_CLK
- U5 pad 39: Net-(U5-DP0N) -> /POWER/~CS
- U5 pad 40: Net-(U5-DP0P) -> unconnected-(U5-GPIO12-Pad40)
- U5 pad 41: GND -> unconnected-(U5-GPIO13-Pad41)
- U5 pad 5: Net-(U5-SSRXP) -> 3V3
- U5 pad 6: Net-(C8-Pad1) -> Net-(U5-ADCIN1)
- U5 pad 7: /USB-C MUX/HUB_SSRX- -> VBUS2
- U5 pad 8: /USB-C MUX/HUB_SSRX+ -> VBUS1
- U5 pad 9: /USB-C MUX/TX1+ -> LDO_3V3
- U6 pad 1: /SD/SWIO -> /POWER/~CS
- U6 pad 2: /SD/DSW1 -> /POWER/D0
- U6 pad 3: GND -> Net-(U6-~{HOLD}/RESET(IO3))
- U6 pad 4: /SD/SD_D- -> GND
- U6 pad 5: /SD/SD_D+ -> /POWER/D1
- U6 pad 6: /SD/3V3 -> /POWER/SPI_CLK
- U6 pad 7: Net-(U6-TXN) -> Net-(U6-~{HOLD}/RESET(IO3))
- U6 pad 8: Net-(U6-TXP) -> LDO_3V3
- U8 pad 1: /USB-C MUX/DP_ML0+ -> DP_ML0+
- U8 pad 2: /USB-C MUX/DP_ML0- -> DP_ML0-
- U8 pad 4: /USB-C MUX/DP_ML1+ -> DP_ML1+
- U8 pad 5: /USB-C MUX/DP_ML1- -> DP_ML1-
- U9 pad 1: /USB-C MUX/USB2*_D- -> TX2+
- U9 pad 2: GND -> TX2-
- U9 pad 3: /USB-C MUX/USB2*_D+ -> GND
- U9 pad 4: /USB-C MUX/USB2_D+ -> RX2+
- U9 pad 5: /USB-C MUX/5V -> RX2-
- U9 pad 6: /USB-C MUX/USB2_D- -> unconnected-(U9-NC-Pad6)
- Y1 pad 1: /USB HUB/XTL0 -> XTL0
- Y1 pad 2: /USB HUB/XTLI -> XTLI
Other:
- board text added: "1V2 LDO"
- board text added: "3V3 Buck"
- board text added: "5V Buck"
- board text added: "PD USB-C"
- board text added: "SPI Flash"

Commit message: Add files via upload
Parts:
- moved C20 94.0 mm to (59.3, 90.1), turned to 180 degrees
- moved R9 80.3 mm to (59.9, 98.1), turned to 180 degrees
- moved R7 79.5 mm to (60.1, 96.0), turned to 180 degrees
- moved U5 76.7 mm to (66.9, 93.7)
- moved C19 75.3 mm to (60.2, 92.2), turned to 180 degrees
- moved R10 73.3 mm to (70.1, 87.8), turned to 90 degrees
- moved C16 72.9 mm to (60.1, 94.0), turned to 180 degrees
- moved R12 70.8 mm to (70.1, 102.7), turned to 90 degrees
- moved C21 70.3 mm to (68.3, 87.9), turned to 90 degrees
- moved R11 68.1 mm to (72.9, 99.6), turned to 90 degrees
- moved C22 66.8 mm to (68.4, 99.5), turned to -90 degrees
- moved C17 61.2 mm to (72.8, 94.0)
- moved C5 1.79 mm to (25.1, 63.0)
- moved R8 1.77 mm to (25.1, 64.6)
- moved C6 1.37 mm to (17.8, 63.9)
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Routing:
- net 3V3: track 0.00 -> 35.8 mm, vias 0 -> 4
- net GND: track 0.00 -> 30.7 mm
- net 5V: track 0.00 -> 26.4 mm, vias 0 -> 2
- net Net-(U2-SW): track 0.00 -> 12.0 mm
- net SYS_PWR: track 0.00 -> 11.5 mm
- net Net-(U6-~{HOLD}/RESET(IO3)): track 0.00 -> 9.80 mm
- net Net-(U1-SW): track 0.00 -> 5.89 mm
- net Net-(U2-FB): track 0.00 -> 4.25 mm
- net LDO_3V3: track 0.00 -> 3.92 mm
- net /POWER/C_CC2(2): track 0.00 -> 3.79 mm, vias 0 -> 1
- net 1V2: track 0.00 -> 3.74 mm, vias 0 -> 1
- net /POWER/CC1(2): track 0.00 -> 3.74 mm, vias 0 -> 1
- net Net-(U1-FB): track 0.00 -> 3.61 mm
- net Net-(U1-EN): track 0.00 -> 2.99 mm
- net Net-(U2-EN): track 0.00 -> 2.96 mm
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- added copper zone on B.Cu, net GND
- added copper zone on F.Cu, net GND
- added copper zone on In1.Cu, net GND
- added copper zone on In2.Cu, net GND
- added copper zone on In3.Cu, net GND
- added copper zone on In4.Cu, net GND
- added copper zone on In5.Cu, net GND
- added copper zone on In6.Cu, net GND
Other:
- copper layers 2 -> 8
